File: unni-smartification-c6/unni-smartification-c6.kicad_pcb (KiCad board)
At the start: 2 copper layers, 83.3 x 65 mm, 72 parts, among them J1 USB-C (replacement daughterbo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, J10 UART TEST, J2 Li-Ion 1S JST-PH, J20 CO2 tap: SDA/SCL/GND, J21 RT/RH tap: RT/RH/GND, J22 TOUCH / LED+ / LED- / GND, J4 UNNI DC / battery input - AC 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, Q1 AO3401A, Q10 AO3400A touch emulator, Q2 AO3401A, Q3 AO3400A, Q4 AO3400A, U1 MCP73831T-2ACI/OT, U10 ESP32-C6-MINI-1, U2 TPS63031DSK, U3 TPS613222ADBZ (5V)

Commit message: Fix PCB net mapping and validate against schematic
Parts:
- added RT1: 10k NTC @25C, Resistor_THT:R_Axial_DIN0204_L3.6mm_D1.6mm_P5.08mm_Horizontal, F.Cu at (0.00, 0.00)
- C1, C2, C3, C5, C6, C7, C8: footprint Capacitor_SMD:C_0805_2012Metric -> Capacitor_SMD:C_0805_2012Metric_Pad1.18x1.45mm_HandSolder
- C10, C11, C12, C13, C20, C21, C30, C31, C32, C33, C4, C9: footprint Capacitor_SMD:C_0603_1608Metric -> Capacitor_SMD:C_0603_1608Metric_Pad1.08x0.95mm_HandSolder
- J1: footprint Connector_USB:USB_C_Receptacle_GCT_USB4105-xx-A_16P_TopMnt_Horizontal -> Misc:SAMESKY_UJ20-C-H-G-SMT-1-P16-TR; moved to B.Cu
- J10, J20, J21, J4: footprint Connector_JST:JST_XH_S3B-XH-A_1x03_P2.50mm_Horizontal -> Connector_JST:JST_PH_S3B-PH-SM4-TB_1x03-1MP_P2.00mm_Horizontal
- J2: footprint Connector_JST:JST_PH_S2B-PH-K_1x02_P2.00mm_Horizontal -> Connector_JST:JST_PH_S2B-PH-SM4-TB_1x02-1MP_P2.00mm_Horizontal
- J22: footprint Connector_JST:JST_XH_S4B-XH-A_1x04_P2.50mm_Horizontal -> Connector_JST:JST_PH_S4B-PH-SM4-TB_1x04-1MP_P2.00mm_Horizontal
- R1, R2: moved to B.Cu
Routing:
- net Net-(J1-CC1): track 0.00 -> 7.64 mm
- net Net-(J1-CC2): track 0.00 -> 7.39 mm
