File: unni-smartification-c6/02_esp_aux.kicad_sch (KiCad schematic)
At the start: 36 parts, among them J10 UART TEST, J20 CO2 tap: SDA/SCL/GND, J21 RT/RH tap: RT/RH/GND, J22 TOUCH / LED+ / LED- / GND, Q10 AO3400A touch emulator, SW1 RESET, SW2 BOOT, U10 ESP32-C6-MINI-1

Commit message: iteration on schematics and simulation
Connections:
- net BACKLIGHT_ADC: no longer C33.1
- net BOOT_GPIO9: now also SW2.2; no longer SW2.1
- net ESP_EN: now also SW1.2; no longer SW1.1
- net GND: now also SW1.1, SW2.1; no longer SW1.2, SW2.2
- net USB_P: now reaches R23.1, U10.18 (IO13)
- net USB_N: now reaches R22.1, U10.17 (IO12)
- net CHARGE_EN: no longer names the net of U10.28 (IO22)
- no-connect marks 11 -> 12
Other:
- moved on the sheet: C10, C11, C12, C30, C31, C32, C33, J20, J21, J22, Q10, R20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

Commit message: Validate power paths and fix KiCad SPICE models
Connections:
- net BACKLIGHT_ADC: now also C33.1
Changed lines of the file:
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@@
 		(title "ESP32-C6 + Auxiliary Circuits")
 		(date "2026-08-19")
-		(rev "A-v28-final")
+		(rev "A-v29-validated")
 		(company "Unni CO2 Smartification")
 	)
@@
 	(wire
 		(pts
-			(xy 309.88 209.55) (xy 309.88 217.17)
-		)
-		(stroke
+			(xy 314.96 209.55) (xy 314.96 217.17)
+		)
+		(stroke
+			(width 0)
+			(type default)
+		)
+	)
+	(wire
+		(pts
+			(xy 314.96 217.17) (xy 309.88 217.17)
+		)
+		(stroke

Commit message: further iterations
Parts:
- R20, R21, R22, R23, R30, R31, R32, R33, R34, R40, R41, R42, R43, R50, R51, R52: footprint Resistor_SMD:R_0603_1608Metric -> Resistor_SMD:R_0805_2012Metric_Pad1.20x1.40mm_HandSolder
Changed lines of the file:
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@@
 	(wire
 		(pts
-			(xy 314.96 217.17) (xy 309.88 217.17)
-		)
-		(stroke
-			(width 0)
-			(type default)
-		)
-	)
-	(wire
-		(pts
 			(xy 210.82 236.22) (xy 210.82 238.76)
 		)
@@
 	(wire
 		(pts
+			(xy 314.96 217.17) (xy 309.88 217.17)
+		)
+		(stroke
+			(width 0)
+			(type default)
+		)
+	)
+	(wire
+		(pts
 			(xy 55.88 148.59) (xy 55.88 156.21)
 		)
@@
 			)
 		)
-		(property "Footprint" "Resistor_SMD:R_0603_1608Metric"
+		(property "Footprint" "Resistor_SMD:R_0805_2012Metric_Pad1.20x1.40mm_HandSolder"
 			(at 320.04 193.04 0)
 			(hide yes)
@@
 			)
 		)
-		(property "Footprint" "Resistor_SMD:R_0603_1608Metric"
+		(property "Footprint" "Resistor_SMD:R_0805_2012Metric_Pad1.20x1.40mm_HandSolder"
 			(at 121.92 137.16 0)
 			(hide yes)
@@
 			)
 		)
-		(property "Footprint" "Resistor_SMD:R_0603_1608Metric"
+		(property "Footprint" "Resistor_SMD:R_0805_2012Metric_Pad1.20x1.40mm_HandSolder"
 			(at 218.44 210.82 0)
 			(hide yes)
@@
 			)
 		)
-		(property "Footprint" "Resistor_SMD:R_0603_1608Metric"
+		(property "Footprint" "Resistor_SMD:R_0805_2012Metric_Pad1.20x1.40mm_HandSolder"
 			(at 40.64 137.16 0)
 			(hide yes)
@@
 			)
 		)
-		(property "Footprint" "Resistor_SMD:R_0603_1608Metric"
+		(property "Footprint" "Resistor_SMD:R_0805_2012Metric_Pad1.20x1.40mm_HandSolder"
 			(at 240.03 73.66 0)
 			(hide yes)
@@
 			)
 		)
-		(property "Footprint" "Resistor_SMD:R_0603_1608Metric"
+		(property "Footprint" "Resistor_SMD:R_0805_2012Metric_Pad1.20x1.40mm_HandSolder"
 			(at 83.82 160.02 0)
 			(hide yes)
@@
 			)
 		)
-		(property "Footprint" "Resistor_SMD:R_0603_1608Metric"
+		(property "Footprint" "Resistor_SMD:R_0805_2012Metric_Pad1.20x1.40mm_HandSolder"
 			(at 218.44 233.68 0)
 			(hide yes)
@@
 			)
 		)
-		(property "Footprint" "Resistor_SMD:R_0603_1608Metric"
+		(property "Footprint" "Resistor_SMD:R_0805_2012Metric_Pad1.20x1.40mm_HandSolder"
 			(at 289.56 219.71 0)
 			(hide yes)
@@
 			)
 		)
-		(property "Footprint" "Resistor_SMD:R_0603_1608Metric"
+		(property "Footprint" "Resistor_SMD:R_0805_2012Metric_Pad1.20x1.40mm_HandSolder"
 			(at 240.03 71.12 0)
 			(hide yes)
@@
 			)
 		)
-		(property "Footprint" "Resistor_SMD:R_0603_1608Metric"
+		(property "Footprint" "Resistor_SMD:R_0805_2012Metric_Pad1.20x1.40mm_HandSolder"
 			(at 218.44 205.74 0)
 			(hide yes)
@@
 			)
 		)
-		(property "Footprint" "Resistor_SMD:R_0603_1608Metric"
+		(property "Footprint" "Resistor_SMD:R_0805_2012Metric_Pad1.20x1.40mm_HandSolder"
 			(at 218.44 238.76 0)
 			(hide yes)
@@
 			)
 		)
-		(property "Footprint" "Resistor_SMD:R_0603_1608Metric"
+		(property "Footprint" "Resistor_SMD:R_0805_2012Metric_Pad1.20x1.40mm_HandSolder"
 			(at 132.08 55.88 0)
 			(hide yes)
@@
 			)
 		)
-		(property "Footprint" "Resistor_SMD:R_0603_1608Metric"
+		(property "Footprint" "Resistor_SMD:R_0805_2012Metric_Pad1.20x1.40mm_HandSolder"
 			(at 40.64 160.02 0)
 			(hide yes)
@@
 			)
 		)
-		(property "Footprint" "Resistor_SMD:R_0603_1608Metric"
+		(property "Footprint" "Resistor_SMD:R_0805_2012Metric_Pad1.20x1.40mm_HandSolder"
 			(at 143.51 83.82 0)
 			(hide yes)
@@
 			)
 		)
-		(property "Footprint" "Resistor_SMD:R_0603_1608Metric"
+		(property "Footprint" "Resistor_SMD:R_0805_2012Metric_Pad1.20x1.40mm_HandSolder"
 			(at 289.56 198.12 0)
 			(hide yes)
@@
 			)
 		)
-		(property "Footprint" "Resistor_SMD:R_0603_1608Metric"
+		(property "Footprint" "Resistor_SMD:R_0805_2012Metric_Pad1.20x1.40mm_HandSolder"
 			(at 83.82 137.16 0)
 			(hide yes)

Commit message: first try doing a pcb with kicad 10.99
Parts:
- J10: footprint Connector_PinHeader_1x03_P2.54mm_Vertical -> Connector_JST:JST_XH_S3B-XH-A_1x03_P2.50mm_Horizontal
- J20, J21: footprint Connector_JST:JST_XH_B3B-XH-A_1x03_P2.50mm_Vertical -> Connector_JST:JST_XH_S3B-XH-A_1x03_P2.50mm_Horizontal
- J22: footprint Connector_JST:JST_XH_B4B-XH-A_1x04_P2.50mm_Vertical -> Connector_JST:JST_XH_S4B-XH-A_1x04_P2.50mm_Horizontal
Changed lines of the file:
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@@
 (kicad_sch
-	(version 20260306)
+	(version 20260818)
 	(generator "eeschema")
-	(generator_version "10.0")
+	(generator_version "10.99")
 	(paper "A3")
 	(title_block
@@
 	)
 	(junction
+		(at 83.82 148.59)
+		(diameter 0)
+		(color 0 0 0 0)
+	)
+	(junction
 		(at 167.64 35.56)
 		(diameter 0)
@@
 	)
 	(junction
+		(at 121.92 148.59)
+		(diameter 0)
+		(color 0 0 0 0)
+	)
+	(junction
+		(at 40.64 148.59)
+		(diameter 0)
+		(color 0 0 0 0)
+	)
+	(junction
 		(at 143.51 91.44)
 		(diameter 0)
@@
 			)
 		)
-		(property "Footprint" "Connector_JST:JST_XH_B4B-XH-A_1x04_P2.50mm_Vertical"
+		(property "Footprint" "Connector_JST:JST_XH_S4B-XH-A_1x04_P2.50mm_Horizontal"
 			(at 279.4 172.72 0)
 			(hide yes)
@@
 			)
 		)
-		(property "Footprint" "Connector_JST:JST_XH_B3B-XH-A_1x03_P2.50mm_Vertical"
+		(property "Footprint" "Connector_JST:JST_XH_S3B-XH-A_1x03_P2.50mm_Horizontal"
 			(at 190.5 236.22 0)
 			(hide yes)
@@
 			)
 		)
-		(property "Footprint" "Connector_PinHeader_1x03_P2.54mm_Vertical"
+		(property "Footprint" "Connector_JST:JST_XH_S3B-XH-A_1x03_P2.50mm_Horizontal"
 			(at 292.1 53.34 0)
 			(hide yes)
@@
 			)
 		)
-		(property "Footprint" "Connector_JST:JST_XH_B3B-XH-A_1x03_P2.50mm_Vertical"
+		(property "Footprint" "Connector_JST:JST_XH_S3B-XH-A_1x03_P2.50mm_Horizontal"
 			(at 190.5 208.28 0)
 			(hide yes)

Commit message: Fix PCB net mapping and validate against schematic
Parts:
- C10, C11, C12, C13, C20, C21, C30, C31, C32, C33: footprint Capacitor_SMD:C_0603_1608Metric -> Capacitor_SMD:C_0603_1608Metric_Pad1.08x0.95mm_HandSolder
- J10, J20, J21: footprint Connector_JST:JST_XH_S3B-XH-A_1x03_P2.50mm_Horizontal -> Connector_JST:JST_PH_S3B-PH-SM4-TB_1x03-1MP_P2.00mm_Horizontal
- J22: footprint Connector_JST:JST_XH_S4B-XH-A_1x04_P2.50mm_Horizontal -> Connector_JST:JST_PH_S4B-PH-SM4-TB_1x04-1MP_P2.00mm_Horizontal
- RT1: footprint Thermistor_SMD:Thermistor_0603_1608Metric -> Resistor_THT:R_Axial_DIN0204_L3.6mm_D1.6mm_P5.08mm_Horizontal
Connections:
- no-connect marks 12 -> 5
Changed lines of the file:
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@@
 	)
 	(no_connect
-		(at 177.8 96.52)
-	)
-	(no_connect
 		(at 175.26 81.28)
 	)
@@
 	)
 	(no_connect
-		(at 203.2 104.14)
-	)
-	(no_connect
-		(at 177.8 99.06)
-	)
-	(no_connect
 		(at 218.44 93.98)
 	)
@@
 		(at 205.74 78.74)
 	)
-	(no_connect
-		(at 203.2 101.6)
-	)
-	(no_connect
-		(at 203.2 99.06)
-	)
-	(no_connect
-		(at 177.8 101.6)
-	)
-	(no_connect
-		(at 177.8 104.14)
-	)
 	(wire
 		(pts
@@
 			)
 		)
-		(property "Footprint" "Connector_JST:JST_XH_S4B-XH-A_1x04_P2.50mm_Horizontal"
+		(property "Footprint" "Connector_JST:JST_PH_S4B-PH-SM4-TB_1x04-1MP_P2.00mm_Horizontal"
 			(at 279.4 172.72 0)
 			(hide yes)
@@
 			)
 		)
-		(property "Footprint" "Capacitor_SMD:C_0603_1608Metric"
+		(property "Footprint" "Capacitor_SMD:C_0603_1608Metric_Pad1.08x0.95mm_HandSolder"
 			(at 55.88 160.02 0)
 			(hide yes)
@@
 			)
 		)
-		(property "Footprint" "Capacitor_SMD:C_0603_1608Metric"
+		(property "Footprint" "Capacitor_SMD:C_0603_1608Metric_Pad1.08x0.95mm_HandSolder"
 			(at 304.8 148.59 0)
 			(hide yes)
@@
 			)
 		)
-		(property "Footprint" "Capacitor_SMD:C_0603_1608Metric"
+		(property "Footprint" "Capacitor_SMD:C_0603_1608Metric_Pad1.08x0.95mm_HandSolder"
 			(at 137.16 160.02 0)
 			(hide yes)
@@
 		(unit 1)
 		(body_style 1)
-		(exclude_from_sim yes)
+		(exclude_from_sim no)
 		(in_bom yes)
 		(on_board yes)
@@
 			(effects
 				(font
-					(size 1 1)
+					(size 1.27 1.27)
 				)
 				(justify left)
@@
 			(effects
 				(font
-					(size 1 1)
+					(size 1.27 1.27)
 				)
 				(justify left)
@@
 		)
 		(property "Footprint" "RF_Module:ESP32-C6-MINI-1"
-			(at 190.5 83.82 0)
+			(at 208.28 109.22 0)
 			(hide yes)
 			(show_name no)
@@
 			(effects
 				(font
-					(size 1 1)
+					(size 1.27 1.27)
 				)
 			)
 		)
-		(property "Datasheet" ""
-			(at 190.5 83.82 0)
+		(property "Datasheet" "https://www.espressif.com/sites/default/files/documentation/esp32-c6-mini-1_mini-1u_datasheet_en.pdf"
+			(at 190.5 46.99 0)
 			(hide yes)
 			(show_name no)
@@
 			(effects
 				(font
-					(size 1 1)
+					(size 1.27 1.27)
 				)
 			)
 		)
-		(property "Description" ""
-			(at 190.5 83.82 0)
+		(property "Description" "RF Module, ESP32-C6 SoC, Wi-Fi 802.11b/g/n/ax, Bluetooth, BLE, Zigbee, Thread, 32-bit, 3.3V, SMD, onboard antenna"
+			(at 190.5 44.45 0)
 			(hide yes)
 			(show_name no)
@@
 			(effects
 				(font
-					(size 1 1)
+					(size 1.27 1.27)
 				)
 			)
 		)
-		(pin "1"
+		(pin "15"
 		)
-		(pin "2"
+		(pin "14"
 		)
-		(pin "3"
+		(pin "32"
 		)
-		(pin "4"
+		(pin "37"
 		)
-		(pin "5"
+		(pin "38"
 		)
-		(pin "6"
+		(pin "33"
 		)
-		(pin "7"
+		(pin "35"
 		)
-		(pin "8"
+		(pin "39"
 		)
-		(pin "9"
+		(pin "40"
 		)
-		(pin "10"
+		(pin "34"
 		)
-		(pin "11"
+		(pin "36"
 		)
-		(pin "12"
+		(pin "41"
 		)
-		(pin "13"
+		(pin "44"
 		)
-		(pin "14"
+		(pin "42"
 		)
-		(pin "15"
+		(pin "45"
 		)
-		(pin "16"
+		(pin "43"
 		)
-		(pin "17"
+		(pin "46"
 		)
-		(pin "18"
+		(pin "50"
 		)
-		(pin "19"
+		(pin "49"
 		)
-		(pin "20"
+		(pin "51"
 		)
-		(pin "21"
+		(pin "47"
 		)
-		(pin "22"
+		(pin "52"
 		)
-		(pin "23"
+		(pin "48"
 		)
-		(pin "24"
+		(pin "53"
 		)
-		(pin "25"
+		(pin "18"
 		)
-		(pin "26"
+		(pin "22"
 		)
-		(pin "27"
+		(pin "19"
 		)
-		(pin "28"
+		(pin "23"
 		)
-		(pin "29"
+		(pin "20"
 		)
-		(pin "30"
+		(pin "21"
 		)
-		(pin "31"
+		(pin "4"
 		)
-		(pin "32"
+		(pin "5"
 		)
-		(pin "33"
+		(pin "8"
 		)
-		(pin "34"
+		(pin "6"
 		)
-		(pin "35"
+		(pin "7"
 		)
-		(pin "36"
+		(pin "11"
 		)
-		(pin "37"
+		(pin "10"
 		)
-		(pin "38"
+		(pin "12"
 		)
-		(pin "39"
+		(pin "13"
 		)
-		(pin "40"
+		(pin "9"
 		)
-		(pin "41"
+		(pin "2"
 		)
-		(pin "42"
+		(pin "3"
 		)
-		(pin "43"
+		(pin "1"
 		)
-		(pin "44"
+		(pin "26"
 		)
-		(pin "45"
+		(pin "24"
 		)
-		(pin "46"
+		(pin "25"
 		)
-		(pin "47"
+		(pin "28"
 		)
-		(pin "48"
+		(pin "29"
 		)
-		(pin "49"
+		(pin "27"
 		)
-		(pin "50"
+		(pin "30"
 		)
-		(pin "51"
+		(pin "31"
 		)
-		(pin "52"
+		(pin "16"
 		)
-		(pin "53"
+		(pin "17"
 		)
 		(instances
@@
 			)
 		)
-		(property "Footprint" "Thermistor_SMD:Thermistor_0603_1608Metric"
+		(property "Footprint" "Resistor_THT:R_Axial_DIN0204_L3.6mm_D1.6mm_P5.08mm_Horizontal"
 			(at 121.92 160.02 0)
 			(hide yes)
@@
 			)
 		)
-		(property "Footprint" "Capacitor_SMD:C_0603_1608Metric"
+		(property "Footprint" "Capacitor_SMD:C_0603_1608Metric_Pad1.08x0.95mm_HandSolder"
 			(at 304.8 163.83 0)
 			(hide yes)
@@
 			)
 		)
-		(property "Footprint" "Connector_JST:JST_XH_S3B-XH-A_1x03_P2.50mm_Horizontal"
+		(property "Footprint" "Connector_JST:JST_PH_S3B-PH-SM4-TB_1x03-1MP_P2.00mm_Horizontal"
 			(at 190.5 236.22 0)
 			(hide yes)
@@
 			)
 		)
-		(property "Footprint" "Connector_JST:JST_XH_S3B-XH-A_1x03_P2.50mm_Horizontal"
+		(property "Footprint" "Connector_JST:JST_PH_S3B-PH-SM4-TB_1x03-1MP_P2.00mm_Horizontal"
 			(at 292.1 53.34 0)
 			(hide yes)
@@
 			)
 		)
-		(property "Footprint" "Capacitor_SMD:C_0603_1608Metric"
+		(property "Footprint" "Capacitor_SMD:C_0603_1608Metric_Pad1.08x0.95mm_HandSolder"
 			(at 156.21 45.72 0)
 			(hide yes)
@@
 			)
 		)
-		(property "Footprint" "Capacitor_SMD:C_0603_1608Metric"
+		(property "Footprint" "Capacitor_SMD:C_0603_1608Metric_Pad1.08x0.95mm_HandSolder"
 			(at 304.8 156.21 0)
 			(hide yes)
@@
 			)
 		)
-		(property "Footprint" "Capacitor_SMD:C_0603_1608Metric"
+		(property "Footprint" "Capacitor_SMD:C_0603_1608Metric_Pad1.08x0.95mm_HandSolder"
 			(at 289.56 81.28 0)
 			(hide yes)
@@
 			)
 		)
-		(property "Footprint" "Connector_JST:JST_XH_S3B-XH-A_1x03_P2.50mm_Horizontal"
+		(property "Footprint" "Connector_JST:JST_PH_S3B-PH-SM4-TB_1x03-1MP_P2.00mm_Horizontal"
 			(at 190.5 208.28 0)
 			(hide yes)
@@
 			)
 		)
-		(property "Footprint" "Capacitor_SMD:C_0603_1608Metric"
+		(property "Footprint" "Capacitor_SMD:C_0603_1608Metric_Pad1.08x0.95mm_HandSolder"
 			(at 167.64 45.72 0)
 			(hide yes)
@@
 			)
 		)
-		(property "Footprint" "Capacitor_SMD:C_0603_1608Metric"
+		(property "Footprint" "Capacitor_SMD:C_0603_1608Metric_Pad1.08x0.95mm_HandSolder"
 			(at 309.88 220.98 0)
 			(hide yes)
@@
 			)
 		)
-		(property "Footprint" "Capacitor_SMD:C_0603_1608Metric"
+		(property "Footprint" "Capacitor_SMD:C_0603_1608Metric_Pad1.08x0.95mm_HandSolder"
 			(at 269.24 83.82 0)
 			(hide yes)

Commit message: trying routing the usb-pcb
Parts:
- Q10: footprint Package_TO_SOT_SMD:SOT-23 -> Package_TO_SOT_SMD:SOT-23_Handsoldering
Changed lines of the file:
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@@
 	(wire
 		(pts
-			(xy 320.04 177.8) (xy 304.8 177.8)
+			(xy 320.04 177.8) (xy 308.61 177.8)
 		)
 		(stroke
@@
 	(global_label "TOUCH_TRIGGER"
 		(shape input)
-		(at 304.8 177.8 180)
+		(at 308.61 177.8 180)
 		(fields_autoplaced yes)
 		(effects
@@
 		)
 		(property "Intersheetrefs" "${INTERSHEET_REFS}"
-			(at 290.6402 177.8 0)
+			(at 294.4502 177.8 0)
 			(hide yes)
 			(show_name no)
@@
 			)
 		)
-		(property "Footprint" "Package_TO_SOT_SMD:SOT-23"
+		(property "Footprint" "Package_TO_SOT_SMD:SOT-23_Handsoldering"
 			(at 335.28 177.8 0)
 			(hide yes)

Commit message: move some power stuff to esp board, update some footprints
Parts:
- added C1, C2: 4.7uF, Capacitor_SMD:C_0805_2012Metric_Pad1.18x1.45mm_HandSolder, symbol Device:C
- added C3, C5, C6: 10uF, Capacitor_SMD:C_0805_2012Metric_Pad1.18x1.45mm_HandSolder, symbol Device:C
- added C4: 100nF, Capacitor_SMD:C_0603_1608Metric_Pad1.08x0.95mm_HandSolder, symbol Device:C
- added D1: SS14, Diode_SMD:D_SMA_Handsoldering, symbol Diode:SB120
- added J2: Li-Ion 1S JST-PH, Connector_JST:JST_PH_S2B-PH-K_1x02_P2.00mm_Horizontal, symbol Connector_Generic:Conn_01x02
- added L1: 2.2uH, Inductor_SMD:L_TDK_NLV32_3.2x2.5mm, symbol Device:L
- added Q1: AO3401A, Package_TO_SOT_SMD:SOT-23_Handsoldering, symbol Transistor_FET:TP0610T
- added R11: 150k, Resistor_SMD:R_0805_2012Metric_Pad1.20x1.40mm_HandSolder, symbol Device:R
- added R12: 220k, Resistor_SMD:R_0805_2012Metric_Pad1.20x1.40mm_HandSolder, symbol Device:R
- added R3: 3.3k, Resistor_SMD:R_0805_2012Metric_Pad1.20x1.40mm_HandSolder, symbol Device:R
- added R5: 100k, Resistor_SMD:R_0805_2012Metric_Pad1.20x1.40mm_HandSolder, symbol Device:R
- added R6: 1M, Resistor_SMD:R_0805_2012Metric_Pad1.20x1.40mm_HandSolder, symbol Device:R
- added U1: MCP73831T-2ACI/OT, Package_TO_SOT_SMD:SOT-23-5_HandSoldering, symbol Battery_Management:MCP73831-2-OT
- added U2: TPS63031DSK, Package_SON:WSON-10-1EP_2.5x2.5mm_P0.5mm_EP1.2x2mm, symbol Regulator_Switching:TPS63030DSK
- SW1, SW2: footprint Button_Switch_SMD:SW_SPST_TL3301AN -> Button_Switch_THT:SW_PUSH_6mm
Connections:
- net +3V3: now also C5.1, C6.1, U2.1 (VOUT), U2.10 (FB)
- net +BATT: now also C2.1, J2.2 (Pin_2), Q1.3 (D), U1.3 (V_{BAT})
- net CHARGE_STAT: now also R11.2, R12.1
- net GND: now also C1.2, C2.2, C3.2, C4.2, C5.2, C6.2, J2.1 (Pin_1), R12.2, R3.2, R6.1, U1.2 (V_{SS}), U2.11 (PGND), U2.3 (PGND), U2.7 (PS/SYNC), U2.9 (GND)
- net VBUS: now also C1.1, D1.2 (A), R5.1, U1.4 (V_{DD})
- new net: R11.1, U1.1 (STAT)
- new net: Q1.1 (G), R5.2, R6.2
- new net: L1.2, U2.2 (L2)
- new net: L1.1, U2.4 (L1)
- new net: R3.1, U1.5 (PROG)
- new net SYS: C3.1, C4.1, D1.1 (K), Q1.2 (S), U2.5 (VIN), U2.6 (EN), U2.8 (VINA)
Other:
- note added: "RPROG 3.3k = ~303 mA nominal charge current"
- moved on the sheet: C10, C11, C12, C13, C20, C21, J10, R20, R21, R22, R23, R30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

Commit message: re-do ESP PCB
Parts:
- removed J10: UART TEST, Connector_JST:JST_PH_S3B-PH-SM4-TB_1x03-1MP_P2.00mm_Horizontal, symbol Connector_Generic:Conn_01x03
- removed J20: CO2 tap: SDA/SCL/GND, Connector_JST:JST_PH_S3B-PH-SM4-TB_1x03-1MP_P2.00mm_Horizontal, symbol Connector_Generic:Conn_01x03
- removed J21: RT/RH tap: RT/RH/GND, Connector_JST:JST_PH_S3B-PH-SM4-TB_1x03-1MP_P2.00mm_Horizontal, symbol Connector_Generic:Conn_01x03
- removed J22: TOUCH / LED+ / LED- / GND, Connector_JST:JST_PH_S4B-PH-SM4-TB_1x04-1MP_P2.00mm_Horizontal, symbol Connector_Generic:Conn_01x04
- removed TP1: BACKLIGHT_LED_NEG, TestPoint:TestPoint_Pad_D1.0mm, symbol Connector:TestPoint
- added J11, J24: Conn_01x01, Connector_Wire:SolderWire-0.5sqmm_1x01_D0.9mm_OD2.1mm, symbol Connector_Generic:Conn_01x01
- added J12, J13, J14, J15, J17, J18, J19, J23, J25, J26, J27: Conn_01x01, Connector_Wire:SolderWire-0.1sqmm_1x01_D0.4mm_OD1mm, symbol Connector_Generic:Conn_01x01
- L1: footprint Inductor_SMD:L_TDK_NLV32_3.2x2.5mm -> Unni_Inductor:L_Murata_LQH3NPN_3.0x3.0mm_HandSolder
- RT1: footprint Resistor_THT:R_Axial_DIN0204_L3.6mm_D1.6mm_P5.08mm_Horizontal -> Connector_PinSocket_2.54mm:PinSocket_1x02_P2.54mm_Vertical
- SW1, SW2: footprint Button_Switch_THT:SW_PUSH_6mm -> Unni_Switch:SW_Jianfu_TVAF36-N014JW-R_HandSolder
Connections:
- net +BATT: now also J27.1 (Pin_1)
- net BOOST_CMD: now also J25.1 (Pin_1)
- net GND: now also J11.1 (Pin_1), J24.1 (Pin_1)
- net VBUS: now also J26.1 (Pin_1)
- net CONN_TOUCH: now reaches C30.1, C31.1, C32.1
- net CONN_TOUCH: now also J14.1 (Pin_1)
- net CONN_LED+: now reaches R50.1
- net CONN_LED+: now also J15.1 (Pin_1)
- net CONN_SCL: now reaches R41.1
- net CONN_SCL: now also J18.1 (Pin_1)
- net CONN_RT: now reaches R42.1
- net CONN_RT: now also J19.1 (Pin_1)
- net CONN_RH: now reaches R43.1
- net CONN_RH: now also J23.1 (Pin_1)
- net CONN_SDA: now reaches R40.1
- net CONN_SDA: now also J17.1 (Pin_1)
- net USB_RAW_N renamed CONN_USB_N
- net CONN_USB_N: now also J12.1 (Pin_1)
- net USB_RAW_P renamed CONN_USB_P
- net CONN_USB_P: now also J13.1 (Pin_1)
- no-connect marks 5 -> 7
