File: unni-smartification-c6/unni-smartification-c6.kicad_sch (KiCad schematic)
At the start: 54 parts, among them J1 Li-ion battery, J2 UNNI DC, J3 CO2 tap, J4 RT/RH tap, J5 Touch/Backlight, J7 USB-C Receptacle, J8 USB daughter -> main, J9 to original UNNI AC, Q1 2N7002, Q2 2N7002, SW1 RESET, SW2 BOOT, U1 ESP32-C6-MINI-1, U2 BQ24074, U3 TPS63031DSK, U4 TPS61023, U5 TPS2116

Commit message: Represent USB data as differential-pair buses
Connections:
- net USB_D+ renamed USB_P
- net USB_D+_RAW renamed USB_RAW_P
- net USB_D- renamed USB_N
- net USB_D-_RAW renamed USB_RAW_N
Other:
- note added: "J8 inter-board pin plan: 1 USB_5V_RAW, 2 USB_RAW_P, 3 USB_RAW_N, 4 UNNI_AC, 5 GND."
- note added: "J8: USB_5V_RAW / USB_RAW_P / USB_RAW_N / UNNI_AC / GND"
- note added: "USB data is represented as KiCad group buses. Nets use *_P/*_N naming so PCB Editor recognizes both sides of R20/R21 as differential pairs. Target USB FS differential impedance: 90 ohm; final width/gap depends on PCB stackup."
- note removed: "J8 inter-board pin plan: 1 USB_5V_RAW, 2 USB_D+_RAW, 3 USB_D-_RAW, 4 UNNI_AC, 5 GND."
- note removed: "J8: USB_5V_RAW / USB_D+ / USB_D- / UNNI_AC / GND"
- note removed: "USB D+/D- between daughterboard and main board route as a 90-ohm differential pair; 22-ohm series resistors are placed close to U1."
Changed lines of the file:
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@@
   (wire (pts (xy 60.24 70.08) (xy 68.00 70.08)) (stroke (width 0) (type default)))
   (wire (pts (xy 68.00 67.54) (xy 68.00 70.08)) (stroke (width 0) (type default)))
-  (global_label "USB_D+_RAW" (shape passive) (at 68.00 68.81 0) (fields_autoplaced yes) (effects (font (size 0.9 0.9)) (justify left)))
+  (global_label "USB_RAW_P" (shape passive) (at 68.00 68.81 0) (fields_autoplaced yes) (effects (font (size 0.9 0.9)) (justify left)))
   (wire (pts (xy 60.24 62.46) (xy 70.00 62.46)) (stroke (width 0) (type default)))
   (wire (pts (xy 60.24 65.00) (xy 70.00 65.00)) (stroke (width 0) (type default)))
   (wire (pts (xy 70.00 62.46) (xy 70.00 65.00)) (stroke (width 0) (type default)))
-  (global_label "USB_D-_RAW" (shape passive) (at 70.00 63.73 0) (fields_autoplaced yes) (effects (font (size 0.9 0.9)) (justify left)))
+  (global_label "USB_RAW_N" (shape passive) (at 70.00 63.73 0) (fields_autoplaced yes) (effects (font (size 0.9 0.9)) (justify left)))
   (symbol (lib_id "Device:R") (at 90.00 92.00 0) (unit 1) (exclude_from_sim no) (in_bom yes) (on_board yes) (dnp no)
     (property "Reference" "R1" (at 90.00 84.00 0) (effects (font (size 1.27 1.27))))
@@
     (instances (project "unni-smartification-c6" (path "/ccd4d3bf-b340-4941-a309-47c78bf5abe8" (reference "J8") (unit 1))))
   )
-  (text "J8: USB_5V_RAW / USB_D+ / USB_D- / UNNI_AC / GND" (exclude_from_sim no) (at 103.00 82.00 0) (effects (font (size 1.0 1.0)) (justify left bottom)))
+  (text "J8: USB_5V_RAW / USB_RAW_P / USB_RAW_N / UNNI_AC / GND" (exclude_from_sim no) (at 103.00 82.00 0) (effects (font (size 1.0 1.0)) (justify left bottom)))
   (wire (pts (xy 109.92 59.92) (xy 102.00 59.92)) (stroke (width 0) (type default)))
   (global_label "USB_5V_RAW" (shape passive) (at 102.00 59.92 180) (fields_autoplaced yes) (effects (font (size 0.9 0.9)) (justify right)))
   (wire (pts (xy 109.92 62.46) (xy 102.00 62.46)) (stroke (width 0) (type default)))
-  (global_label "USB_D+_RAW" (shape passive) (at 102.00 62.46 180) (fields_autoplaced yes) (effects (font (size 0.9 0.9)) (justify right)))
+  (global_label "USB_RAW_P" (shape passive) (at 102.00 62.46 180) (fields_autoplaced yes) (effects (font (size 0.9 0.9)) (justify right)))
   (wire (pts (xy 109.92 65.00) (xy 102.00 65.00)) (stroke (width 0) (type default)))
-  (global_label "USB_D-_RAW" (shape passive) (at 102.00 65.00 180) (fields_autoplaced yes) (effects (font (size 0.9 0.9)) (justify right)))
+  (global_label "USB_RAW_N" (shape passive) (at 102.00 65.00 180) (fields_autoplaced yes) (effects (font (size 0.9 0.9)) (justify right)))
   (wire (pts (xy 109.92 67.54) (xy 102.00 67.54)) (stroke (width 0) (type default)))
   (global_label "UNNI_AC" (shape passive) (at 102.00 67.54 180) (fields_autoplaced yes) (effects (font (size 0.9 0.9)) (justify right)))
@@
   (global_label "BOOST_EN" (shape passive) (at 363.24 95.08 0) (fields_autoplaced yes) (effects (font (size 0.9 0.9)) (justify left)))
   (wire (pts (xy 355.24 77.30) (xy 363.24 77.30)) (stroke (width 0) (type default)))
-  (global_label "USB_D-" (shape passive) (at 363.24 77.30 0) (fields_autoplaced yes) (effects (font (size 0.9 0.9)) (justify left)))
+  (global_label "USB_N" (shape passive) (at 363.24 77.30 0) (fields_autoplaced yes) (effects (font (size 0.9 0.9)) (justify left)))
   (wire (pts (xy 355.24 79.84) (xy 363.24 79.84)) (stroke (width 0) (type default)))
-  (global_label "USB_D+" (shape passive) (at 363.24 79.84 0) (fields_autoplaced yes) (effects (font (size 0.9 0.9)) (justify left)))
+  (global_label "USB_P" (shape passive) (at 363.24 79.84 0) (fields_autoplaced yes) (effects (font (size 0.9 0.9)) (justify left)))
   (wire (pts (xy 355.24 72.22) (xy 363.24 72.22)) (stroke (width 0) (type default)))
   (global_label "UART_RX" (shape passive) (at 363.24 72.22 0) (fields_autoplaced yes) (effects (font (size 0.9 0.9)) (justify left)))
@@
     (instances (project "unni-smartification-c6" (path "/6233a2c5-4e5d-493d-9a56-a8751a784ff1" (reference "R20") (unit 1))))
   )
-  (global_label "USB_D-_RAW" (shape passive) (at 310.00 161.19 0) (fields_autoplaced yes) (effects (font (size 0.9 0.9)) (justify left)))
-  (global_label "USB_D-" (shape passive) (at 310.00 168.81 180) (fields_autoplaced yes) (effects (font (size 0.9 0.9)) (justify right)))
+  (global_label "USB_RAW_N" (shape passive) (at 310.00 161.19 0) (fields_autoplaced yes) (effects (font (size 0.9 0.9)) (justify left)))
+  (global_label "USB_N" (shape passive) (at 310.00 168.81 180) (fields_autoplaced yes) (effects (font (size 0.9 0.9)) (justify right)))
   (symbol (lib_id "Device:R") (at 330.00 165.00 0) (unit 1) (exclude_from_sim no) (in_bom yes) (on_board yes) (dnp no)
     (property "Reference" "R21" (at 330.00 157.00 0) (effects (font (size 1.27 1.27))))
@@
     (instances (project "unni-smartification-c6" (path "/0c0e50d6-2cdc-44cb-a7c4-23c4f207f153" (reference "R21") (unit 1))))
   )
-  (global_label "USB_D+_RAW" (shape passive) (at 330.00 161.19 0) (fields_autoplaced yes) (effects (font (size 0.9 0.9)) (justify left)))
-  (global_label "USB_D+" (shape passive) (at 330.00 168.81 180) (fields_autoplaced yes) (effects (font (size 0.9 0.9)) (justify right)))
-  (text "USB D+/D- between daughterboard and main board route as a 90-ohm differential pair; 22-ohm series resistors are placed close to U1." (exclude_from_sim no) (at 300.00 178.00 0) (effects (font (size 1.0 1.0)) (justify left bottom)))
-  (text "J8 inter-board pin plan: 1 USB_5V_RAW, 2 USB_D+_RAW, 3 USB_D-_RAW, 4 UNNI_AC, 5 GND." (exclude_from_sim no) (at 20.00 122.00 0) (effects (font (size 1.0 1.0)) (justify left bottom)))
+  (global_label "USB_RAW_P" (shape passive) (at 330.00 161.19 0) (fields_autoplaced yes) (effects (font (size 0.9 0.9)) (justify left)))
+  (global_label "USB_P" (shape passive) (at 330.00 168.81 180) (fields_autoplaced yes) (effects (font (size 0.9 0.9)) (justify right)))
+  (bus (pts (xy 295.91 181.61) (xy 344.17 181.61)) (stroke (width 0) (type default)))
+  (label "{USB_RAW_P USB_RAW_N}" (at 295.91 181.61 0) (effects (font (size 0.9 0.9)) (justify left bottom)))
+  (bus (pts (xy 295.91 185.42) (xy 344.17 185.42)) (stroke (width 0) (type default)))
+  (label "{USB_P USB_N}" (at 295.91 185.42 0) (effects (font (size 0.9 0.9)) (justify left bottom)))
+  (text "USB data is represented as KiCad group buses. Nets use *_P/*_N naming so PCB Editor recognizes both sides of R20/R21 as differential pairs. Target USB FS differential impedance: 90 ohm; final width/gap depends on PCB stackup." (exclude_from_sim no) (at 300.00 178.00 0) (effects (font (size 1.0 1.0)) (justify left bottom)))
+  (text "J8 inter-board pin plan: 1 USB_5V_RAW, 2 USB_RAW_P, 3 USB_RAW_N, 4 UNNI_AC, 5 GND." (exclude_from_sim no) (at 20.00 122.00 0) (effects (font (size 1.0 1.0)) (justify left bottom)))
   (text "J9 original-Unni connection: UNNI_AC + GND. Main-board J2: VBAT/UNNI_DC + GND." (exclude_from_sim no) (at 20.00 127.00 0) (effects (font (size 1.0 1.0)) (justify left bottom)))
   (sheet_instances (path "/" (page "1")))

Commit message: Wire complete functional blocks explicitly
Connections:
- net ILIM_NODE is gone; now on an unnamed net: U2.12 (ILIM)
- net BOOST_5V: now also U4.1 (FB); no longer C10.1, C9.1, R8.1
- net GND: now also R3.2, R4.2, R5.1; no longer C1.2, C10.2, C2.2, C4.2, C5.2, C6.2, C8.2, C9.2, R9.2, U2.17 (EP), U2.4 (CE), U2.8 (VSS), U3.11 (PGND), U3.3 (PGND), U3.9 (GND)
- net SYS: no longer U3.8 (VINA)
- net TOUCH_RAW: no longer C11.1, C12.1, C13.1
- net UNNI_AC: no longer U5.2 (VOUT), U5.7 (VOUT)
- net USB_5V_RAW: no longer C1.1, U2.13 (IN), U5.4 (PR1), U5.5 (MODE)
- net USB_RAW_N: no longer J7.A7 (D-), J7.B7 (D-)
- net USB_RAW_P: no longer J7.A6 (D+), J7.B6 (D+)
- net VBAT: no longer L2.1
- net BB_L1: no longer names the net of L1.1, U3.4 (L1)
- net BB_L2: no longer names the net of L1.2, U3.2 (L2)
- net BOOST_FB: no longer names the net of R8.2, R9.1
- net BOOST_FB: no longer U4.1 (FB)
- net BOOST_SW: no longer names the net of U4.5 (SW)
- net BOOST_SW: now also L2.1; no longer L2.2
- net CO2_SCL_RAW: no longer names the net of J3.2 (Pin_2), R11.1
- net CO2_SDA_RAW: no longer names the net of J3.1 (Pin_1), R10.1
- net ISET_NODE: no longer names the net of U2.16 (ISET)
- net RH_RAW: no longer names the net of J4.2 (Pin_2), R13.1
- net RT_RAW: no longer names the net of J4.1 (Pin_1), R12.1
- removed net TOUCH_SW: C11.2, C12.2, C13.2
- net TS_NODE: no longer names the net of U2.1 (TS)
- new net: U5.2 (VOUT), U5.7 (VOUT)
- new net: U5.4 (PR1), U5.5 (MODE)
- new net: J7.A6 (D+), J7.B6 (D+)
- new net: J7.A7 (D-), J7.B7 (D-)
- new net: C10.2, C8.2
- new net: U3.11 (PGND), U3.3 (PGND)
Other:
- note added: "Q1 / BOOST_EN_HW is the hardware-inhibit stage; final polarity/gate conditioning will be checked in ERC/design review."
- note added: "TPS2116: VIN1 USB_5V_RAW has priority over VIN2 BOOST_5V; both VOUT pins are visibly tied to UNNI_AC."
- note added: "TPS63031 fixed 3.3 V: FB is visibly tied to VOUT; PS/SYNC is wired low for power-save."
- note added: "USB / LI-ION CHARGER + POWERPATH — BQ24074"
- note added: "USB D+/D-: the schematic bus groups the pair; the 22-ohm series resistors are shown inline and are placed close to U1."
- note removed: "Hardware inhibit: USB_5V_RAW forces BOOST_EN_HW low. BOOST_EN from ESP can only enable boost when external USB is absent."
- note removed: "TPS2116 priority mode: VIN1=USB_5V_RAW, VIN2=BOOST_5V, VOUT=UNNI_AC. Reverse-current blocking prevents boost backfeed into USB."
- note removed: "TPS63031 fixed 3.3 V: FB tied to VOUT; PS/SYNC low = power-save. 1.5 uH + 10 uF input + 2x10 uF output."
- note removed: "USB / LI-ION POWER PATH"
- note removed: "USB data is represented as KiCad group buses. Nets use *_P/*_N naming so PCB Editor recognizes both sides of R20/R21 as differential pairs. Target USB FS differential impedance: 90 ohm; final width/gap depends on PCB stackup."

Commit message: chatgpt refines the schematic
Parts:
- removed C1: 4.7uF, Capacitor_SMD:C_0603_1608Metric, symbol Device:C
- removed C10, C9: 22uF, Capacitor_SMD:C_0603_1608Metric, symbol Device:C
- removed C2, C3, C8: 10uF, Capacitor_SMD:C_0603_1608Metric, symbol Device:C
- removed J1: Li-ion battery, Connector_JST:JST_PH_B2B-PH-K_1x02_P2.00mm_Vertical, symbol Connector_Generic:Conn_01x02
- removed J2: UNNI DC, Connector_JST:JST_XH_B2B-XH-A_1x02_P2.50mm_Vertical, symbol Connector_Generic:Conn_01x02
- removed L2: 1.0uH, Inductor_SMD:L_Changjiang_FNR3015S, symbol Device:L
- removed Q1: 2N7002, Package_TO_SOT_SMD:SOT-23, symbol UNNI:2N7002
- removed R3: 3.0k, Resistor_SMD:R_0603_1608Metric, symbol Device:R
- removed R4: 1.18k, Resistor_SMD:R_0603_1608Metric, symbol Device:R
- removed R5: 10k, Resistor_SMD:R_0603_1608Metric, symbol Device:R
- removed R8: 732k, Resistor_SMD:R_0603_1608Metric, symbol Device:R
- removed R9: 100k, Resistor_SMD:R_0603_1608Metric, symbol Device:R
- removed U2: BQ24074, Package_DFN_QFN:VQFN-16-1EP_3x3mm_P0.5mm_EP1.68x1.68mm, symbol UNNI:BQ24074
- removed U4: TPS61023, Package_SOT:SOT-563, symbol UNNI:TPS61023
- removed U5: TPS2116, Package_SOT:SOT-563-8, symbol UNNI:TPS2116
- added C101, C102: 1uF, Capacitor_SMD:C_0603_1608Metric, symbol Device:C
- added C103: 10uF, Capacitor_SMD:C_0805_2012Metric, symbol Device:C
- added C104: 22uF, Capacitor_SMD:C_0805_2012Metric, symbol Device:C
- added C105: 100nF, Capacitor_SMD:C_0603_1608Metric, symbol Device:C
- added D101: SS14, Diode_SMD:D_SMA, symbol Device:D_Schottky
- added D102: DNP / SS14, Diode_SMD:D_SMA, symbol Device:D_Schottky
- added L101: 2.2uH, Inductor_SMD:L_1210_3225Metric, symbol Device:L
- added Q101, Q102: AO3401A, Package_TO_SOT_SMD:SOT-23, symbol Transistor_FET:Q_PMOS_GSD
- added Q103, Q104: AO3400A, Package_TO_SOT_SMD:SOT-23, symbol Transistor_FET:Q_NMOS_GSD
- added R101: 3.3k, Resistor_SMD:R_0603_1608Metric, symbol Device:R
- added R102, R103, R106, R107: 100k, Resistor_SMD:R_0603_1608Metric, symbol Device:R
- added R104, R108, R110, R111: 1M, Resistor_SMD:R_0603_1608Metric, symbol Device:R
- added R105, R114: 10k, Resistor_SMD:R_0603_1608Metric, symbol Device:R
- added R112, R113: 220k, Resistor_SMD:R_0603_1608Metric, symbol Device:R
- added R115: 10k NTC, Resistor_SMD:R_0603_1608Metric, symbol Device:R
- added U101: MCP73812T-420I/OT, Package_TO_SOT_SMD:SOT-23-5, symbol Battery_Management:MCP73812T-420I-OT
- added U102: TPS613222ADBZ, Package_TO_SOT_SMD:SOT-23, symbol Regulator_Switching:TPS613222ADBZ
- added U103, U104: AP22913W6-7, Package_TO_SOT_SMD:SOT-23-6, symbol Power_Management:AP22913CN4
Connections:
- net USB_5V_RAW is gone; now on net GND: J7.A4 (VBUS), J7.A9 (VBUS), J7.B4 (VBUS), J7.B9 (VBUS), J8.1 (Pin_1), R18.1
- net BAT_ADC: now also R110.2, R111.1
- net BOOST_5V: now also U104.B2 (ON)
- net GND: now also C101.1, C101.2, C102.2, C103.2, C104.2, C105.2, Q101.1 (G), Q102.1 (G), Q103.2 (S), Q103.3 (D), Q104.1 (G), Q104.3 (D), R101.1, R102.2, R103.1, R103.2, R104.1, R104.2, R106.2, R107.2, R108.1, R108.2, R111.2, R112.1, R113.2, R115.2, U101.2 (V_{SS}), U101.4 (V_{DD}), U103.B2 (ON)
- net SYS: now also Q101.2 (S)
- net USB_ADC: now also R112.2, R113.1
- net USB_N: now also U1.29 (IO23); no longer U1.17 (IO12)
- net USB_P: now also U1.28 (IO22); no longer U1.18 (IO13)
- net VBAT: now also C102.1, Q101.3 (D), Q102.3 (D), R106.1, R110.1
- net CHARGE_EN: now reaches U1.19 (IO14)
- net CHARGE_EN: now also R102.1, U101.5 (PROG)
- net BAT_TEMP_ADC: now reaches U1.27 (IO21)
- net BAT_TEMP_ADC: now also R114.2, R115.1
- new net: Q103.1 (G), Q104.2 (S), R105.2, R107.1
- new net: R101.2, U101.1 (CE)
- new net BAT_TEMP_EXCITE: C105.1, R114.1, U1.18 (IO13)
- new net BOOST_CMD: R105.1, U1.17 (IO12)
- new net BOOST_VIN: C103.1, L101.1, Q102.2 (S)
- no-connect marks 11 -> 8
Other:
- note added: "ADC SENSE + BATTERY TEMPERATURE"
- note added: "FORCED-AWAKE 5 V — TPS613222A + AO3401/AO3400 INHIBIT + AP22913 OR-ING"
- note added: "Q101: 100k from USB to gate + 1M gate pulldown. USB present -> PMOS off; USB absent -> battery path on."
- note added: "TPS613222A is hard-disconnected in normal battery mode. Q104 forces BOOST_GATE low whenever real USB is present."
- note added: "U103/U104 are AP22913 logical symbols; PCB target is AP22913W6-7 SOT-26. OFF-state TRCB prevents backfeed between real USB and boosted 5 V."
- note added: "UNNI CO2 SMARTIFICATION — REV A / ESP32-C6-MINI-1 — LOW-COST POWER"
- note added: "USB / LI-ION CHARGER + LOAD SHARING — MCP73812 + AO3401A"
- note added: "~300 mA charge. CE is MCU-controlled and defaults low. USB feeds SYS through Schottky; battery feeds SYS through Q101 only when USB is absent."
- note removed: "FORCED-AWAKE 5 V + USB PRIORITY MUX"
- note removed: "J8 inter-board pin plan: 1 USB_5V_RAW, 2 USB_RAW_P, 3 USB_RAW_N, 4 UNNI_AC, 5 GND."
- note removed: "J9 original-Unni connection: UNNI_AC + GND. Main-board J2: VBAT/UNNI_DC + GND."
- note removed: "Q1 / BOOST_EN_HW is the hardware-inhibit stage; final polarity/gate conditioning will be checked in ERC/design review."
- note removed: "TPS2116: VIN1 USB_5V_RAW has priority over VIN2 BOOST_5V; both VOUT pins are visibly tied to UNNI_AC."
- note removed: "UNNI CO2 SMARTIFICATION — REV A / ESP32-C6-MINI-1"
- note removed: "USB / LI-ION CHARGER + POWERPATH — BQ24074"
- note removed: "VBAT is the battery node and is also routed directly to UNNI_DC."

Commit message: schematic sheets & spice
Parts:
- removed C101, C102: 1uF, Capacitor_SMD:C_0603_1608Metric, symbol Device:C
- removed C103: 10uF, Capacitor_SMD:C_0805_2012Metric, symbol Device:C
- removed C104: 22uF, Capacitor_SMD:C_0805_2012Metric, symbol Device:C
- removed C105, C5: 100nF, Capacitor_SMD:C_0603_1608Metric, symbol Device:C
- removed C11: 47pF, Capacitor_SMD:C_0603_1608Metric, symbol Device:C
- removed C12: 100pF, Capacitor_SMD:C_0603_1608Metric, symbol Device:C
- removed C13: 220pF, Capacitor_SMD:C_0603_1608Metric, symbol Device:C
- removed C14: 10nF DNP, Capacitor_SMD:C_0603_1608Metric, symbol Device:C
- removed C4, C6, C7: 10uF, Capacitor_SMD:C_0603_1608Metric, symbol Device:C
- removed D101: SS14, Diode_SMD:D_SMA, symbol Device:D_Schottky
- removed D102: DNP / SS14, Diode_SMD:D_SMA, symbol Device:D_Schottky
- removed J3: CO2 tap, Connector_JST:JST_XH_B3B-XH-A_1x03_P2.50mm_Vertical, symbol Connector_Generic:Conn_01x03
- removed J4: RT/RH tap, Connector_JST:JST_XH_B3B-XH-A_1x03_P2.50mm_Vertical, symbol Connector_Generic:Conn_01x03
- removed J5: Touch/Backlight, Connector_JST:JST_XH_B4B-XH-A_1x04_P2.50mm_Vertical, symbol Connector_Generic:Conn_01x04
- removed J7: USB-C Receptacle, Connector_USB:USB_C_Receptacle_GCT_USB4105-xx-A_16P_TopMnt_Horizontal, symbol Connector:USB_C_Receptacle_USB2.0_16P
- removed J8: USB daughter -> main, Connector_JST:JST_XH_B5B-XH-A_1x05_P2.50mm_Vertical, symbol Connector_Generic:Conn_01x05
- removed J9: to original UNNI AC, Connector_JST:JST_XH_B2B-XH-A_1x02_P2.50mm_Vertical, symbol Connector_Generic:Conn_01x02
- removed L1: 1.5uH, Inductor_SMD:L_Changjiang_FNR3015S, symbol Device:L
- removed L101: 2.2uH, Inductor_SMD:L_1210_3225Metric, symbol Device:L
- removed Q101, Q102: AO3401A, Package_TO_SOT_SMD:SOT-23, symbol Transistor_FET:Q_PMOS_GSD
- removed Q103, Q104: AO3400A, Package_TO_SOT_SMD:SOT-23, symbol Transistor_FET:Q_NMOS_GSD
- removed Q2: 2N7002, Package_TO_SOT_SMD:SOT-23, symbol UNNI:2N7002
- removed R1, R2: 5.1k, Resistor_SMD:R_0603_1608Metric, symbol Device:R
- removed R10, R105, R11, R114, R12, R13, R6, R7: 10k, Resistor_SMD:R_0603_1608Metric, symbol Device:R
- removed R101: 3.3k, Resistor_SMD:R_0603_1608Metric, symbol Device:R
- removed R102, R103, R106, R107: 100k, Resistor_SMD:R_0603_1608Metric, symbol Device:R
- removed R104, R108, R110, R111, R16, R17: 1M, Resistor_SMD:R_0603_1608Metric, symbol Device:R
- removed R112, R113, R15, R18, R19: 220k, Resistor_SMD:R_0603_1608Metric, symbol Device:R
- removed R115: 10k NTC, Resistor_SMD:R_0603_1608Metric, symbol Device:R
- removed R14: 330k, Resistor_SMD:R_0603_1608Metric, symbol Device:R
- removed R20, R21: 22R, Resistor_SMD:R_0402_1005Metric, symbol Device:R
- removed SW1: RESET, Button_Switch_SMD:SW_SPST_PTS810, symbol UNNI:SW_Push
- removed SW2: BOOT, Button_Switch_SMD:SW_SPST_PTS810, symbol UNNI:SW_Push
- removed U1: ESP32-C6-MINI-1, RF_Module:ESP32-C6-MINI-1, symbol RF_Module:ESP32-C6-MINI-1
- removed U101: MCP73812T-420I/OT, Package_TO_SOT_SMD:SOT-23-5, symbol Battery_Management:MCP73812T-420I-OT
- removed U102: TPS613222ADBZ, Package_TO_SOT_SMD:SOT-23, symbol Regulator_Switching:TPS613222ADBZ
- removed U103, U104: AP22913W6-7, Package_TO_SOT_SMD:SOT-23-6, symbol Power_Management:AP22913CN4
- removed U3: TPS63031DSK, Package_SON:WSON-10-1EP_2.5x2.5mm_P0.5mm_EP1.2x2mm, symbol Regulator_Switching:TPS63031DSK
Connections:
- no-connect marks 8 -> 0
Other:
- added sheet ESP32-C6 + Auxiliary (02_esp_aux.kicad_sch)
- added sheet USB + Power (01_usb_power.kicad_sch)
- note added: "Two-sheet cleanup: standard power symbols, grid-aligned wiring, explicit local connectivity."
- note added: "UNNI CO2 SMARTIFICATION — REV A"
- note removed: "3.3 V ESP SUPPLY — TPS63031 BUCK-BOOST"
- note removed: "ADC SENSE"
- note removed: "ADC SENSE + BATTERY TEMPERATURE"
- note removed: "All Unni signal connections are T-taps. Removing the smartification PCB leaves the original Unni signal paths untouched."
- note removed: "ESP32-C6-MINI-1 + NATIVE USB"
- note removed: "FORCED-AWAKE 5 V — TPS613222A + AO3401/AO3400 INHIBIT + AP22913 OR-ING"
- note removed: "Flat schematic intentionally used for Rev A validation. Functional blocks are separated visually; all inter-block nets use named global labels."
- note removed: "GPIO4/5/8/9/15 are strapping pins; Rev A avoids them for Unni runtime signals except GPIO9 used only as BOOT."
- note removed: "J8: USB_5V_RAW / USB_RAW_P / USB_RAW_N / UNNI_AC / GND"
- note removed: "Q101: 100k from USB to gate + 1M gate pulldown. USB present -> PMOS off; USB absent -> battery path on."
- note removed: "REPLACEMENT USB-C DAUGHTERBOARD"
- note removed: "Replacement daughterboard keeps the original case USB-C opening; smartification board returns muxed UNNI_AC here."
- note removed: "TPS613222A is hard-disconnected in normal battery mode. Q104 forces BOOST_GATE low whenever real USB is present."
- note removed: "TPS63031 fixed 3.3 V: FB is visibly tied to VOUT; PS/SYNC is wired low for power-save."
- note removed: "U103/U104 are AP22913 logical symbols; PCB target is AP22913W6-7 SOT-26. OFF-state TRCB prevents backfeed between real USB and boosted 5 V."
- note removed: "UNNI CO2 SMARTIFICATION — REV A / ESP32-C6-MINI-1 — LOW-COST POWER"
- note removed: "UNNI PASSIVE SIGNAL TAPS + TOUCH/BACKLIGHT"
- note removed: "USB / LI-ION CHARGER + LOAD SHARING — MCP73812 + AO3401A"
- note removed: "USB D+/D-: the schematic bus groups the pair; the 22-ohm series resistors are shown inline and are placed close to U1."
- note removed: "~300 mA charge. CE is MCU-controlled and defaults low. USB feeds SYS through Schottky; battery feeds SYS through Q101 only when USB is absent."
