File: unni-smartification-c6/01_usb_power.kicad_sch (KiCad schematic)
At the start: 21 parts, among them J1 USB-C (replacement daughterbo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, J3 Conn_01x06, J4 UNNI DC / battery input - AC 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, Q2 AO3401A, Q3 AO3400A, Q4 AO3400A, U3 TPS613222ADBZ (5V), U4 TPD2E009DBZR

Commit message: redid some routing, add btn for manual measurements from unni
Parts:
- J3: now not fitted
Changed lines of the file:
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@@
 		(on_board yes)
 		(in_pos_files yes)
-		(dnp no)
+		(dnp yes)
 		(fields_autoplaced yes)
 		(property "Reference" "J3"

Commit message: Add BOM Metadata, iBom, fix validation, pcbway order
this is the state the PCBs were ordered at PCBWay.com

Thank you PCBWay for sponsoring the boards for this ridicoulus project!
Parts:
- C7: Manufacturer (none) -> Samsung Electro-Mechanics; Manufacturer Part Number (none) -> CL21A106KAYNNNE; TME Link (none) -> https://www.tme.eu/de/katalog/?search=CL21A106KAYNNNE; TME Part Number (none) -> CL21A106KAYNNNE
- C8: Manufacturer (none) -> Samsung Electro-Mechanics; Manufacturer Part Number (none) -> CL21A226KPCLRNC; TME Link (none) -> https://www.tme.eu/de/katalog/?search=CL21A226KPCLRNC; TME Part Number (none) -> CL21A226KPCLRNC
- C9: Manufacturer (none) -> Samsung Electro-Mechanics; Manufacturer Part Number (none) -> CL10A105KB8NNNC; TME Link (none) -> https://www.tme.eu/de/katalog/?search=CL10A105KB8NNNC; TME Part Number (none) -> CL10A105KB8NNNC
- D2: Manufacturer (none) -> onsemi; Manufacturer Part Number (none) -> SS14; TME Link (none) -> https://www.tme.eu/en/details/ss14-fai/smd-schottky-diodes/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; TME Part Number (none) -> SS14-FAI
- D3: value SS14 USB -> UNNI_AC -> SS14; Manufacturer (none) -> onsemi; Manufacturer Part Number (none) -> SS14; TME Link (none) -> https://www.tme.eu/en/details/ss14-fai/smd-schottky-diodes/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; TME Part Number (none) -> SS14-FAI
- D4: value SS14 BOOST -> UNNI_AC -> SS14; Manufacturer (none) -> onsemi; Manufacturer Part Number (none) -> SS14; TME Link (none) -> https://www.tme.eu/en/details/ss14-fai/smd-schottky-diodes/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; TME Part Number (none) -> SS14-FAI
- J1: value USB-C (replacement daughterboard) -> UJ20-C-H-G-SMT-1-P16-TR; MANUFACTURER Same Sky -> (none); Manufacturer (none) -> Same Sky; Manufacturer Part Number (none) -> UJ20-C-H-G-SMT-1-P16-TR; TME Link (none) -> https://www.tme.eu/de/katalog/?search=UJ20-C-H-G-SMT-1-P16-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; TME Part Number (none) -> N/A — not listed at TME
- J3: value Conn_01x06 -> B6B-PH-K-S; Manufacturer (none) -> JST; Manufacturer Part Number (none) -> B6B-PH-K-S (LF)(SN); TME Link (none) -> https://www.tme.eu/de/details/b6b-ph-k-s/signalsteckverbind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; TME Part Number (none) -> B6B-PH-K-S
- J4: value UNNI DC / battery input - AC / 5V Input -> S3B-PH-SM4-TB; Manufacturer (none) -> JST; Manufacturer Part Number (none) -> S3B-PH-SM4-TB(LF)(SN); TME Link (none) -> https://www.tme.eu/de/katalog/?search=S3B-PH-SM4-TB; TME Part Number (none) -> S3B-PH-SM4-TB
- L2: Manufacturer (none) -> Murata; Manufacturer Part Number (none) -> DFE322520FD-2R2M=P2; TME Link (none) -> https://www.tme.eu/en/details/dfe322520fd-2r2m/inductors/mu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; TME Part Number (none) -> DFE322520FD-2R2M
- Q2: Manufacturer (none) -> Alpha & Omega Semiconductor; Manufacturer Part Number (none) -> AO3401A; TME Link (none) -> https://www.tme.eu/de/details/ao3401a/p-kanal-transistoren-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; TME Part Number (none) -> AO3401A
- Q3, Q4: Manufacturer (none) -> Alpha & Omega Semiconductor; Manufacturer Part Number (none) -> AO3400A; TME Link (none) -> https://www.tme.eu/de/details/ao3400a/n-kanal-transistoren-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; TME Part Number (none) -> AO3400A
- R1, R2: Manufacturer (none) -> Yageo; Manufacturer Part Number (none) -> RC0805FR-075K1L; TME Link (none) -> https://www.tme.eu/de/katalog/?search=RC0805FR-075K1L; TME Part Number (none) -> RC0805FR-075K1
- R13: Manufacturer (none) -> Yageo; Manufacturer Part Number (none) -> RC0805FR-0747KL; TME Link (none) -> https://www.tme.eu/de/katalog/?search=RC0805FR-0747KL; TME Part Number (none) -> RC0805FR-0747K
- R7, R9: Manufacturer (none) -> Yageo; Manufacturer Part Number (none) -> RC0805FR-071ML; TME Link (none) -> https://www.tme.eu/de/katalog/?search=RC0805FR-071ML; TME Part Number (none) -> RC0805FR-071M
- R8: Manufacturer (none) -> Yageo; Manufacturer Part Number (none) -> RC0805FR-0710KL; TME Link (none) -> https://www.tme.eu/de/katalog/?search=RC0805FR-0710KL; TME Part Number (none) -> RC0805FR-0710K
- U3: value TPS613222ADBZ (5V) -> TPS613222A; Manufacturer (none) -> Texas Instruments; Manufacturer Part Number (none) -> TPS613222ADBZR; TME Link (none) -> https://www.tme.eu/de/katalog/?search=TPS613222ADBZR; TME Part Number (none) -> N/A — not listed at TME
- U4: Manufacturer (none) -> Texas Instruments; Manufacturer Part Number (none) -> TPD2E009DBZR; TME Link (none) -> https://www.tme.eu/en/details/tpd2e009dbzr/protection-diode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; TME Part Number (none) -> TPD2E009DBZR

Commit message: update PCB layout a bit
Parts:
- U3: value TPS613222A -> TPS613222ADBV; footprint Package_TO_SOT_SMD:SOT-23_Handsoldering -> Package_TO_SOT_SMD:SOT-23-5; symbol Regulator_Switching:TPS613221ADBZ -> Regulator_Switching:TPS613222ADBV
Connections:
- net +5V: now also U3.4 (VOUT); no longer U3.1 (VOUT)
- net GND: now also U3.2 (GND); no longer U3.3 (GND)
- net at D2.2 (A), L2.2: now also U3.1 (SW); no longer U3.2 (SW)
Changed lines of the file:
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@@
 	)
 	(symbol
-		(lib_id "Regulator_Switching:TPS613221ADBZ")
+		(lib_id "Regulator_Switching:TPS613222ADBV")
 		(at 133.35 176.53 0)
 		(unit 1)
@@
 			)
 		)
-		(property "Value" "TPS613222A"
+		(property "Value" "TPS613222ADBV"
 			(at 133.35 168.91 0)
 			(show_name no)
@@
 			(effects
 				(font
-					(size 1 1)
+					(size 1.27 1.27)
 				)
 			)
 		)
-		(property "Footprint" "Package_TO_SOT_SMD:SOT-23_Handsoldering"
-			(at 133.35 176.53 0)
+		(property "Footprint" "Package_TO_SOT_SMD:SOT-23-5"
+			(at 133.35 196.85 0)
 			(hide yes)
 			(show_name no)
@@
 			(effects
 				(font
-					(size 1 1)
+					(size 1.27 1.27)
 				)
 			)
 		)
-		(property "Datasheet" "https://www.ti.com/lit/ds/symlink/tps61322.pdf"
-			(at 133.35 176.53 0)
+		(property "Datasheet" "http://www.ti.com/lit/ds/symlink/tps61322.pdf"
+			(at 133.35 180.34 0)
 			(hide yes)
 			(show_name no)
@@
 			(effects
 				(font
-					(size 1 1)
+					(size 1.27 1.27)
 				)
 			)
 		)
-		(property "Description" ""
+		(property "Description" "1.8A Step-Up Converter, 5V Output Voltage, 0.9-5.5V Input Voltage, SOT-23-5"
 			(at 133.35 176.53 0)
 			(hide yes)
@@
 			(effects
 				(font
-					(size 1 1)
+					(size 1.27 1.27)
 				)
 			)
@@
 		(pin "3"
 		)
+		(pin "4"
+		)
+		(pin "5"
+		)
 		(instances
 			(project "unni-smartification-c6"
@@
 		)
 	)
+	(group "5V Boost TPS613222ADBZ"
+		(lib_id "Library:5V Boost TPS613222ADBZ")
+		(members "01083c63-ba25-48c9-b27b-caf93458f60c" "04c9d2d5-f6e0-457d-b9be-a52cb7061d7d"
+			"05126eed-77df-4554-a978-4ec69a96e79b" "0e50fb23-d8f3-4991-8067-e55211285e55"
+			"115efad9-6298-44f2-aa10-6d75fd4ff61f" "12413106-fa23-44df-8048-e91d618386cb"
+			"1493afe2-607a-4734-8e31-3f808e15ecf6" "14947983-38b7-453a-a70c-76cd76293bed"
+			"2782b409-f722-493f-817d-d19e4de81822" "2ac8d321-7c89-41e5-a576-3bbb20dec863"
+			"38b2c436-f720-4723-b82a-04b91d6fe175" "4fb8006e-102e-4671-9c77-b450670fc563"
+			"504901ea-5195-4545-97d2-df4407ae09a3" "51d7401e-9223-40c8-8cac-4c48839b2e79"
+			"538b046a-09b1-4f31-9f83-7d2ff4ecef04" "5e0443d0-ea60-416a-b7e0-c40577ad85ac"
+			"5e519403-d5e2-442b-a7b7-6a2702a99b26" "8811a838-4a51-4921-b7fe-d5a8c1f248f1"
+			"8d363c4f-8d48-4a7d-bf1a-5390f2e986e8" "9364f048-a019-4715-9b4e-02b856920780"
+			"9cb2dc49-ee52-4b21-9f79-3fa642389efb" "aa3a111e-7031-4fe6-a139-95f801208e81"
+			"ac46210f-2e14-4170-8925-16b7b04e7bc6" "acc4ef8e-a949-4554-bb17-fa6a2d11e6d1"
+			"acf80f90-2a82-40e3-bf4d-2e13f0e6eb89" "b6431ef4-80eb-46aa-8cc8-419584bbc460"
+			"c329f727-e446-486f-90e4-c2f2e63b8b46" "c47244fc-cc71-41bf-8938-1b75fb7e414f"
+			"ce398a50-4c81-4c08-8619-b4b77ecd2f8c" "d2b9675a-f727-45bc-aefc-fee8eb43deff"
+			"e72f689f-73b0-4a0c-a0bc-7f7d403a89ad" "f2a256d2-afe4-4e30-ada0-56618362332c"
+			"fbdb7a1d-dd4e-46cf-8e39-5485571848cb"
+		)
+	)
 	(group "USB-PD-5V-ESD"
 		(lib_id "Library:USB-PD-5V-ESD")
@@
 	(group "5V Boost TPS613222ADBZ"
 		(lib_id "Library:5V Boost TPS613222ADBZ")
-		(members "01083c63-ba25-48c9-b27b-caf93458f60c" "04c9d2d5-f6e0-457d-b9be-a52cb7061d7d"
-			"05126eed-77df-4554-a978-4ec69a96e79b" "0e50fb23-d8f3-4991-8067-e55211285e55"
-			"115efad9-6298-44f2-aa10-6d75fd4ff61f" "12413106-fa23-44df-8048-e91d618386cb"
-			"1493afe2-607a-4734-8e31-3f808e15ecf6" "14947983-38b7-453a-a70c-76cd76293bed"
-			"2782b409-f722-493f-817d-d19e4de81822" "2ac8d321-7c89-41e5-a576-3bbb20dec863"
-			"38b2c436-f720-4723-b82a-04b91d6fe175" "4fb8006e-102e-4671-9c77-b450670fc563"
-			"504901ea-5195-4545-97d2-df4407ae09a3" "51d7401e-9223-40c8-8cac-4c48839b2e79"
-			"538b046a-09b1-4f31-9f83-7d2ff4ecef04" "5e0443d0-ea60-416a-b7e0-c40577ad85ac"
-			"5e519403-d5e2-442b-a7b7-6a2702a99b26" "8811a838-4a51-4921-b7fe-d5a8c1f248f1"
-			"8d363c4f-8d48-4a7d-bf1a-5390f2e986e8" "9364f048-a019-4715-9b4e-02b856920780"
-			"9cb2dc49-ee52-4b21-9f79-3fa642389efb" "aa3a111e-7031-4fe6-a139-95f801208e81"
-			"ac46210f-2e14-4170-8925-16b7b04e7bc6" "acc4ef8e-a949-4554-bb17-fa6a2d11e6d1"
-			"acf80f90-2a82-40e3-bf4d-2e13f0e6eb89" "b6431ef4-80eb-46aa-8cc8-419584bbc460"
-			"c329f727-e446-486f-90e4-c2f2e63b8b46" "c47244fc-cc71-41bf-8938-1b75fb7e414f"
-			"ce398a50-4c81-4c08-8619-b4b77ecd2f8c" "d2b9675a-f727-45bc-aefc-fee8eb43deff"
-			"e72f689f-73b0-4a0c-a0bc-7f7d403a89ad" "f2a256d2-afe4-4e30-ada0-56618362332c"
-			"fbdb7a1d-dd4e-46cf-8e39-5485571848cb"
-		)
+		(members "7a10a620-9f61-44f1-b32c-2b571210db2c")
 	)
 )
