File: unni-smartification-c6/dist/kicad-10.0.5/unni-smartification-c6/01_usb_power.kicad_sch (KiCad schematic)
At the start: 21 parts, among them J1 USB-C (replacement daughterbo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, J3 Conn_01x06, J4 UNNI DC / battery input - AC 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, Q2 AO3401A, Q3 AO3400A, Q4 AO3400A, U3 TPS613222ADBZ (5V), U4 TPD2E009DBZR

Commit message: redid some routing, add btn for manual measurements from unni
Parts:
- J3: now not fitted
Changed lines of the file:
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@@
 		(on_board yes)
 		(in_pos_files yes)
-		(dnp no)
+		(dnp yes)
 		(fields_autoplaced yes)
 		(property "Reference" "J3"

Commit message: Add BOM Metadata, iBom, fix validation, pcbway order
this is the state the PCBs were ordered at PCBWay.com

Thank you PCBWay for sponsoring the boards for this ridicoulus project!
Parts:
- C7: Manufacturer (none) -> Samsung Electro-Mechanics; Manufacturer Part Number (none) -> CL21A106KAYNNNE; TME Link (none) -> https://www.tme.eu/de/katalog/?search=CL21A106KAYNNNE; TME Part Number (none) -> CL21A106KAYNNNE
- C8: Manufacturer (none) -> Samsung Electro-Mechanics; Manufacturer Part Number (none) -> CL21A226KPCLRNC; TME Link (none) -> https://www.tme.eu/de/katalog/?search=CL21A226KPCLRNC; TME Part Number (none) -> CL21A226KPCLRNC
- C9: Manufacturer (none) -> Samsung Electro-Mechanics; Manufacturer Part Number (none) -> CL10A105KB8NNNC; TME Link (none) -> https://www.tme.eu/de/katalog/?search=CL10A105KB8NNNC; TME Part Number (none) -> CL10A105KB8NNNC
- D2: Manufacturer (none) -> onsemi; Manufacturer Part Number (none) -> SS14; TME Link (none) -> https://www.tme.eu/en/details/ss14-fai/smd-schottky-diodes/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; TME Part Number (none) -> SS14-FAI
- D3: value SS14 USB -> UNNI_AC -> SS14; Manufacturer (none) -> onsemi; Manufacturer Part Number (none) -> SS14; TME Link (none) -> https://www.tme.eu/en/details/ss14-fai/smd-schottky-diodes/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; TME Part Number (none) -> SS14-FAI
- D4: value SS14 BOOST -> UNNI_AC -> SS14; Manufacturer (none) -> onsemi; Manufacturer Part Number (none) -> SS14; TME Link (none) -> https://www.tme.eu/en/details/ss14-fai/smd-schottky-diodes/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; TME Part Number (none) -> SS14-FAI
- J1: value USB-C (replacement daughterboard) -> UJ20-C-H-G-SMT-1-P16-TR; MANUFACTURER Same Sky -> (none); Manufacturer (none) -> Same Sky; Manufacturer Part Number (none) -> UJ20-C-H-G-SMT-1-P16-TR; TME Link (none) -> https://www.tme.eu/de/katalog/?search=UJ20-C-H-G-SMT-1-P16-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; TME Part Number (none) -> N/A — not listed at TME
- J3: value Conn_01x06 -> B6B-PH-K-S; Manufacturer (none) -> JST; Manufacturer Part Number (none) -> B6B-PH-K-S (LF)(SN); TME Link (none) -> https://www.tme.eu/de/details/b6b-ph-k-s/signalsteckverbind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; TME Part Number (none) -> B6B-PH-K-S
- J4: value UNNI DC / battery input - AC / 5V Input -> S3B-PH-SM4-TB; Manufacturer (none) -> JST; Manufacturer Part Number (none) -> S3B-PH-SM4-TB(LF)(SN); TME Link (none) -> https://www.tme.eu/de/katalog/?search=S3B-PH-SM4-TB; TME Part Number (none) -> S3B-PH-SM4-TB
- L2: Manufacturer (none) -> Murata; Manufacturer Part Number (none) -> DFE322520FD-2R2M=P2; TME Link (none) -> https://www.tme.eu/en/details/dfe322520fd-2r2m/inductors/mu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; TME Part Number (none) -> DFE322520FD-2R2M
- Q2: Manufacturer (none) -> Alpha & Omega Semiconductor; Manufacturer Part Number (none) -> AO3401A; TME Link (none) -> https://www.tme.eu/de/details/ao3401a/p-kanal-transistoren-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; TME Part Number (none) -> AO3401A
- Q3, Q4: Manufacturer (none) -> Alpha & Omega Semiconductor; Manufacturer Part Number (none) -> AO3400A; TME Link (none) -> https://www.tme.eu/de/details/ao3400a/n-kanal-transistoren-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; TME Part Number (none) -> AO3400A
- R1, R2: Manufacturer (none) -> Yageo; Manufacturer Part Number (none) -> RC0805FR-075K1L; TME Link (none) -> https://www.tme.eu/de/katalog/?search=RC0805FR-075K1L; TME Part Number (none) -> RC0805FR-075K1
- R13: Manufacturer (none) -> Yageo; Manufacturer Part Number (none) -> RC0805FR-0747KL; TME Link (none) -> https://www.tme.eu/de/katalog/?search=RC0805FR-0747KL; TME Part Number (none) -> RC0805FR-0747K
- R7, R9: Manufacturer (none) -> Yageo; Manufacturer Part Number (none) -> RC0805FR-071ML; TME Link (none) -> https://www.tme.eu/de/katalog/?search=RC0805FR-071ML; TME Part Number (none) -> RC0805FR-071M
- R8: Manufacturer (none) -> Yageo; Manufacturer Part Number (none) -> RC0805FR-0710KL; TME Link (none) -> https://www.tme.eu/de/katalog/?search=RC0805FR-0710KL; TME Part Number (none) -> RC0805FR-0710K
- U3: value TPS613222ADBZ (5V) -> TPS613222A; Manufacturer (none) -> Texas Instruments; Manufacturer Part Number (none) -> TPS613222ADBZR; TME Link (none) -> https://www.tme.eu/de/katalog/?search=TPS613222ADBZR; TME Part Number (none) -> N/A — not listed at TME
- U4: Manufacturer (none) -> Texas Instruments; Manufacturer Part Number (none) -> TPD2E009DBZR; TME Link (none) -> https://www.tme.eu/en/details/tpd2e009dbzr/protection-diode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; TME Part Number (none) -> TPD2E009DBZR
