File: unni-smartification-c6/dist/kicad-10.0.5/unni-smartification-c6/02_esp_aux.kicad_sch (KiCad schematic)
At the start: 50 parts, among them J10 Conn_01x06, J2 Li-Ion 1S JST-PH, J5 Conn_01x02, J6 Conn_01x05, Q1 AO3401A, Q10 AO3400A touch emulator, SW1 RESET, SW2 BOOT, U1 MCP73831T-2ACI/OT, U10 ESP32-C6-MINI-1, U2 TPS63031DSK

Commit message: redid some routing, add btn for manual measurements from unni
Parts:
- J5: footprint Connector_JST:JST_PH_B2B-PH-K_1x02_P2.00mm_Vertical -> Connector_JST:JST_PH_B3B-PH-K_1x03_P2.00mm_Vertical; symbol Connector_Generic:Conn_01x02 -> Connector_Generic:Conn_01x03
Connections:
- net CONN_BTN: now reaches U10.28 (IO22)
- net CONN_BTN: now also J5.3 (Pin_3)
- no-connect marks 7 -> 5
Changed lines of the file:
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@@
 	)
 	(no_connect
-		(at 267.97 76.2)
-	)
-	(no_connect
 		(at 267.97 68.58)
 	)
 	(no_connect
-		(at 267.97 66.04)
-	)
-	(no_connect
-		(at 311.15 81.28)
+		(at 298.45 66.04)
 	)
 	(no_connect
-		(at 298.45 66.04)
+		(at 267.97 66.04)
 	)
 	(no_connect
@@
 		)
 	)
+	(global_label "CONN_LED+"
+		(shape input)
+		(at 82.55 199.39 180)
+		(fields_autoplaced yes)
+		(effects
+			(font
+				(size 1 1)
+			)
+			(justify right)
+		)
+		(property "Intersheetrefs" "${INTERSHEET_REFS}"
+			(at 71.3426 199.39 0)
+			(hide yes)
+			(show_name no)
+			(do_not_autoplace no)
+			(effects
+				(font
+					(size 1.27 1.27)
+				)
+				(justify right)
+			)
+		)
+	)
 	(global_label "GND"
 		(shape input)
@@
 		)
 	)
-	(global_label "CONN_LED+"
+	(global_label "CONN_TOUCH"
 		(shape input)
-		(at 82.55 201.93 180)
+		(at 82.55 196.85 180)
 		(fields_autoplaced yes)
 		(effects
@@
 		)
 		(property "Intersheetrefs" "${INTERSHEET_REFS}"
-			(at 71.3426 201.93 0)
+			(at 70.3903 196.85 0)
 			(hide yes)
 			(show_name no)
@@
 		)
 	)
+	(global_label "CONN_BTN"
+		(shape input)
+		(at 82.55 201.93 180)
+		(fields_autoplaced yes)
+		(effects
+			(font
+				(size 1 1)
+			)
+			(justify right)
+		)
+		(property "Intersheetrefs" "${INTERSHEET_REFS}"
+			(at 72.4855 201.93 0)
+			(hide yes)
+			(show_name no)
+			(do_not_autoplace no)
+			(effects
+				(font
+					(size 1.27 1.27)
+				)
+				(justify right)
+			)
+		)
+	)
+	(global_label "CONN_BTN"
+		(shape input)
+		(at 311.15 81.28 0)
+		(fields_autoplaced yes)
+		(effects
+			(font
+				(size 1 1)
+			)
+			(justify left)
+		)
+		(property "Intersheetrefs" "${INTERSHEET_REFS}"
+			(at 321.2145 81.28 0)
+			(hide yes)
+			(show_name no)
+			(do_not_autoplace no)
+			(effects
+				(font
+					(size 1.27 1.27)
+				)
+				(justify left)
+			)
+		)
+	)
 	(global_label "CONN_RH"
 		(shape input)
@@
 		)
 	)
-	(global_label "CONN_TOUCH"
-		(shape input)
-		(at 82.55 199.39 180)
-		(fields_autoplaced yes)
-		(effects
-			(font
-				(size 1 1)
-			)
-			(justify right)
-		)
-		(property "Intersheetrefs" "${INTERSHEET_REFS}"
-			(at 70.3903 199.39 0)
-			(hide yes)
-			(show_name no)
-			(do_not_autoplace no)
-			(effects
-				(font
-					(size 1.27 1.27)
-				)
-				(justify right)
-			)
-		)
-	)
 	(global_label "BAT_TEMP_EXCITE"
 		(shape output)
@@
 	)
 	(symbol
-		(lib_id "Connector_Generic:Conn_01x02")
+		(lib_id "Connector_Generic:Conn_01x03")
 		(at 87.63 199.39 0)
 		(unit 1)
 		(body_style 1)
-		(exclude_from_sim yes)
+		(exclude_from_sim no)
 		(in_bom yes)
 		(on_board yes)
@@
 		(fields_autoplaced yes)
 		(property "Reference" "J5"
-			(at 90.17 199.3899 0)
+			(at 90.17 198.1199 0)
 			(show_name no)
 			(do_not_autoplace no)
@@
 		)
 		(property "Value" "Conn_01x02"
-			(at 90.17 201.9299 0)
+			(at 90.17 200.6599 0)
 			(show_name no)
 			(do_not_autoplace no)
@@
 			)
 		)
-		(property "Footprint" "Connector_JST:JST_PH_B2B-PH-K_1x02_P2.00mm_Vertical"
+		(property "Footprint" "Connector_JST:JST_PH_B3B-PH-K_1x03_P2.00mm_Vertical"
 			(at 87.63 199.39 0)
 			(hide yes)
@@
 			)
 		)
-		(property "Description" "Generic connector, single row, 01x02, script generated (kicad-library-utils/schlib/autogen/connector/)"
+		(property "Description" "Generic connector, single row, 01x03, script generated (kicad-library-utils/schlib/autogen/connector/)"
 			(at 87.63 199.39 0)
 			(hide yes)
@@
 		(pin "1"
 		)
+		(pin "3"
+		)
 		(instances

Commit message: Prepare Rev A prototype and add PCBWay sponsorship
Parts:
- C32: value 220pF DNP -> 220pF
- J5: value Conn_01x02 -> Conn_01x03
Connections:
- no-connect marks 5 -> 6
Changed lines of the file:
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@@
 	)
 	(no_connect
+		(at 267.97 76.2)
+	)
+	(no_connect
 		(at 298.45 50.8)
 	)
@@
 			)
 		)
-		(property "Value" "220pF DNP"
+		(property "Value" "220pF"
 			(at 304.8 171.45 90)
 			(show_name no)
@@
 		(unit 1)
 		(body_style 1)
-		(exclude_from_sim no)
+		(exclude_from_sim yes)
 		(in_bom yes)
 		(on_board yes)
@@
 			)
 		)
-		(property "Value" "Conn_01x02"
+		(property "Value" "Conn_01x03"
 			(at 90.17 200.6599 0)
 			(show_name no)

Commit message: Add BOM Metadata, iBom, fix validation, pcbway order
this is the state the PCBs were ordered at PCBWay.com

Thank you PCBWay for sponsoring the boards for this ridicoulus project!
Parts:
- added R24: 10K, Resistor_SMD:R_0603_1608Metric_Pad0.98x0.95mm_HandSolder, symbol Device:R
- C1, C2: Manufacturer (none) -> Samsung Electro-Mechanics; Manufacturer Part Number (none) -> CL21A475KAQNNNE; TME Link (none) -> https://www.tme.eu/de/katalog/?search=CL21A475KAQNNNE; TME Part Number (none) -> CL21A475KAQNNNE
- C10: Manufacturer (none) -> Samsung Electro-Mechanics; Manufacturer Part Number (none) -> CL10A106MQ8NNNC; TME Link (none) -> https://www.tme.eu/de/katalog/?search=CL10A106MQ8NNNC; TME Part Number (none) -> CL10A106MQ8NNNC
- C11, C20, C21, C22, C4: Manufacturer (none) -> Samsung Electro-Mechanics; Manufacturer Part Number (none) -> CL10B104KB8NNNC; TME Link (none) -> https://www.tme.eu/de/katalog/?search=CL10B104KB8NNNC; TME Part Number (none) -> CL10B104KB8NNNC
- C12, C13: Manufacturer (none) -> Samsung Electro-Mechanics; Manufacturer Part Number (none) -> CL10C220JB8NNNC; TME Link (none) -> https://www.tme.eu/de/katalog/?search=CL10C220JB8NNNC; TME Part Number (none) -> CL10C220JB8NNNC
- C3, C5, C6: Manufacturer (none) -> Samsung Electro-Mechanics; Manufacturer Part Number (none) -> CL21A106KAYNNNE; TME Link (none) -> https://www.tme.eu/de/katalog/?search=CL21A106KAYNNNE; TME Part Number (none) -> CL21A106KAYNNNE
- C32: Manufacturer (none) -> Samsung Electro-Mechanics; Manufacturer Part Number (none) -> CL10B221KB8NNNC; TME Link (none) -> https://www.tme.eu/de/katalog/?search=CL10B221KB8NNNC; TME Part Number (none) -> CL10B221KB8NNNC
- C33: Manufacturer (none) -> Samsung Electro-Mechanics; Manufacturer Part Number (none) -> CL10B103KB8NNNC; TME Link (none) -> https://www.tme.eu/de/katalog/?search=CL10B103KB8NNNC; TME Part Number (none) -> CL10B103KB8NNNC
- D1: Manufacturer (none) -> onsemi; Manufacturer Part Number (none) -> SS14; TME Link (none) -> https://www.tme.eu/en/details/ss14-fai/smd-schottky-diodes/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; TME Part Number (none) -> SS14-FAI
- J10: value Conn_01x06 -> B6B-PH-K-S; Manufacturer (none) -> JST; Manufacturer Part Number (none) -> B6B-PH-K-S (LF)(SN); TME Link (none) -> https://www.tme.eu/de/details/b6b-ph-k-s/signalsteckverbind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; TME Part Number (none) -> B6B-PH-K-S
- J2: value Li-Ion 1S JST-PH -> B2B-PH-K-S; Manufacturer (none) -> JST; Manufacturer Part Number (none) -> B2B-PH-K-S (LF)(SN); TME Link (none) -> https://www.tme.eu/de/details/b2b-ph-k-s/signalsteckverbind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; TME Part Number (none) -> B2B-PH-K-S
- J5: value Conn_01x03 -> B3B-PH-K-S; Manufacturer (none) -> JST; Manufacturer Part Number (none) -> B3B-PH-K-S (LF)(SN); TME Link (none) -> https://www.tme.eu/de/details/b3b-ph-k-s/signalsteckverbind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; TME Part Number (none) -> B3B-PH-K-S
- J6: value Conn_01x05 -> B5B-PH-K-S; Manufacturer (none) -> JST; Manufacturer Part Number (none) -> B5B-PH-K-S (LF)(SN); TME Link (none) -> https://www.tme.eu/de/details/b5b-ph-k-s/signalsteckverbind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; TME Part Number (none) -> B5B-PH-K-S
- L1: Manufacturer (none) -> Murata; Manufacturer Part Number (none) -> LQH3NPN2R2MJRL; TME Link (none) -> https://www.tme.eu/en/details/lqh3npn2r2mjrl/inductors/mura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; TME Part Number (none) -> LQH3NPN2R2MJRL
- Q1: Manufacturer (none) -> Alpha & Omega Semiconductor; Manufacturer Part Number (none) -> AO3401A; TME Link (none) -> https://www.tme.eu/de/details/ao3401a/p-kanal-transistoren-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; TME Part Number (none) -> AO3401A
- Q10: value AO3400A touch emulator -> AO3400A; Manufacturer (none) -> Alpha & Omega Semiconductor; Manufacturer Part Number (none) -> AO3400A; TME Link (none) -> https://www.tme.eu/de/details/ao3400a/n-kanal-transistoren-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; TME Part Number (none) -> AO3400A
- R11: Manufacturer (none) -> Yageo; Manufacturer Part Number (none) -> RC0805FR-07150KL; TME Link (none) -> https://www.tme.eu/de/katalog/?search=RC0805FR-07150KL; TME Part Number (none) -> RC0805FR-07150K
- R12, R32, R33, R51: Manufacturer (none) -> Yageo; Manufacturer Part Number (none) -> RC0805FR-07220KL; TME Link (none) -> https://www.tme.eu/de/katalog/?search=RC0805FR-07220KL; TME Part Number (none) -> RC0805FR-07220K
- R20, R21, R34: Manufacturer (none) -> Yageo; Manufacturer Part Number (none) -> RC0805FR-0710KL; TME Link (none) -> https://www.tme.eu/de/katalog/?search=RC0805FR-0710KL; TME Part Number (none) -> RC0805FR-0710K
- R22, R23: Manufacturer (none) -> Yageo; Manufacturer Part Number (none) -> RC0805FR-0722RL; TME Link (none) -> https://www.tme.eu/de/katalog/?search=RC0805FR-0722RL; TME Part Number (none) -> RC0805FR-0722R
- R3: Manufacturer (none) -> Yageo; Manufacturer Part Number (none) -> RC0805FR-075K1L; TME Link (none) -> https://www.tme.eu/de/katalog/?search=RC0805FR-075K1L; TME Part Number (none) -> RC0805FR-075K1
- R30, R31, R6: Manufacturer (none) -> Yageo; Manufacturer Part Number (none) -> RC0805FR-071ML; TME Link (none) -> https://www.tme.eu/de/katalog/?search=RC0805FR-071ML; TME Part Number (none) -> RC0805FR-071M
- R40, R41, R42, R43: Manufacturer (none) -> Yageo; Manufacturer Part Number (none) -> RC0603FR-0710KL; TME Link (none) -> https://www.tme.eu/de/katalog/?search=RC0603FR-0710KL; TME Part Number (none) -> RC0603FR-0710K
- R5, R52: Manufacturer (none) -> Yageo; Manufacturer Part Number (none) -> RC0805FR-07100KL; TME Link (none) -> https://www.tme.eu/de/katalog/?search=RC0805FR-07100KL; TME Part Number (none) -> RC0805FR-07100K
- R50: Manufacturer (none) -> Yageo; Manufacturer Part Number (none) -> RC0805FR-07330KL; TME Link (none) -> https://www.tme.eu/de/katalog/?search=RC0805FR-07330KL; TME Part Number (none) -> RC0805FR-07330K
- RT1: value 10k NTC @25C -> NTCC-10K; Manufacturer (none) -> SR Passives; Manufacturer Part Number (none) -> NTCC-10K; TME Link (none) -> https://www.tme.eu/de/details/ntcc-10k/ntc-mess-thermistore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; TME Part Number (none) -> NTCC-10K
- SW1, SW2: Manufacturer (none) -> Jianfu; Manufacturer Part Number (none) -> TVAF36-N014JW-R; TME Link (none) -> https://www.tme.eu/gb/details/tvaf36n014jwr/microswitches-t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; TME Part Number (none) -> TVAF36N014JWR
- U1: value MCP73831T-2ACI/OT -> MCP73831; Manufacturer (none) -> Microchip Technology; Manufacturer Part Number (none) -> MCP73831T-2ACI/OT; TME Link (none) -> https://www.tme.eu/de/details/mcp73831t-2aci_ot/batterie-u-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; TME Part Number (none) -> MCP73831T-2ACI/OT
- U10: value ESP32-C6-MINI-1 -> ESP32-C6-MINI-1-N4; Manufacturer (none) -> Espressif Systems; Manufacturer Part Number (none) -> ESP32-C6-MINI-1-N4; TME Link (none) -> https://www.tme.eu/de/details/esp32-c6-mini-1-n4/iot-wifi-b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; TME Part Number (none) -> ESP32-C6-MINI-1-N4
- U2: value TPS63031DSK -> TPS63031; Manufacturer (none) -> Texas Instruments; Manufacturer Part Number (none) -> TPS63031DSKR; TME Link (none) -> https://www.tme.eu/en/details/tps63031dskr/voltage-regulato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; TME Part Number (none) -> TPS63031DSKR
Connections:
- net CONN_BTN: now also R24.2; no longer U10.28 (IO22)
- new net: R24.1, U10.28 (IO22)
