File: unni-smartification-c6/dist/kicad-10.0.5/unni-smartification-c6/experimental/unni-smartification-c6-10.99-constraints.kicad_pcb (KiCad board)
At the start: 2 copper layers, 19 x 18 mm, 77 parts, among them J1 USB-C (replacement daughterbo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, J2 Li-Ion 1S JST-PH, J20 CO2 tap: SDA/SCL/GND, J21 RT/RH tap: RT/RH/GND, J22 TOUCH / LED+ / LED- / GND, J3 UNNI AC / 5V input, J4 UNNI DC / battery input, Q1 AO3401A, Q10 AO3400A touch emulator, Q2 AO3401A, Q3 AO3400A, Q4 AO3400A, U1 MCP73831T-2ACI/OT, U10 ESP32-C6-MINI-1, U2 TPS63031DSK, U3 TPS613222ADBZ (5V)

Commit message: Add BOM Metadata, iBom, fix validation, pcbway order
this is the state the PCBs were ordered at PCBWay.com

Thank you PCBWay for sponsoring the boards for this ridicoulus project!
Parts:
- C32: value 220pF DNP -> 220pF
- D3: value SS14 USB -> UNNI_AC -> SS14
- D4: value SS14 BOOST -> UNNI_AC -> SS14
- J1: value USB-C (replacement daughterboard) -> UJ20-C-H-G-SMT-1-P16-TR
- J2: value Li-Ion 1S JST-PH -> B2B-PH-K-S
- J3: value UNNI AC / 5V input -> B6B-PH-K-S
- J4: value UNNI DC / battery input -> S3B-PH-SM4-TB
- Q10: value AO3400A touch emulator -> AO3400A
- R3: value 3.3k -> 5.1k
- R9: value 100k -> 1M
- U1: value MCP73831T-2ACI/OT -> MCP73831
- U10: value ESP32-C6-MINI-1 -> ESP32-C6-MINI-1-N4
- U2: value TPS63031DSK -> TPS63031
- U3: value TPS613222ADBZ (5V) -> TPS613222A
Changed lines of the file:
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@@
 			)
 		)
-		(property "Value" "UNNI DC / battery input"
+		(property "Value" "S3B-PH-SM4-TB"
 			(at 1.25 4.6 0)
 			(layer "F.Fab")
@@
 			)
 		)
-		(property "Value" "TPS63031DSK"
+		(property "Value" "TPS63031"
 			(at 0 2.2 0)
 			(layer "F.Fab")
@@
 			)
 		)
-		(property "Value" "UNNI AC / 5V input"
+		(property "Value" "B6B-PH-K-S"
 			(at 1.25 4.6 0)
 			(layer "F.Fab")
@@
 			)
 		)
-		(property "Value" "TPS613222ADBZ (5V)"
+		(property "Value" "TPS613222A"
 			(at 0 2.4 0)
 			(layer "F.Fab")
@@
 			)
 		)
-		(property "Value" "100k"
+		(property "Value" "1M"
 			(at 0 1.43 0)
 			(layer "F.Fab")
@@
 			)
 		)
-		(property "Value" "SS14 USB -> UNNI_AC"
+		(property "Value" "SS14"
 			(at 0 2.6 0)
 			(layer "F.Fab")
@@
 			)
 		)
-		(property "Value" "Li-Ion 1S JST-PH"
+		(property "Value" "B2B-PH-K-S"
 			(at 1 4 0)
 			(layer "F.Fab")
@@
 			)
 		)
-		(property "Value" "USB-C (replacement daughterboard)"
+		(property "Value" "UJ20-C-H-G-SMT-1-P16-TR"
 			(at 0 5 180)
 			(unlocked yes)
@@
 			)
 		)
-		(property "Value" "220pF DNP"
+		(property "Value" "220pF"
 			(at 0 1.43 90)
 			(layer "F.Fab")
@@
 			)
 		)
-		(property "Value" "AO3400A touch emulator"
+		(property "Value" "AO3400A"
 			(at 0 2.4 90)
 			(layer "F.Fab")
@@
 			)
 		)
-		(property "Value" "MCP73831T-2ACI/OT"
+		(property "Value" "MCP73831"
 			(at 0 2.4 0)
 			(layer "F.Fab")
@@
 			)
 		)
-		(property "Value" "ESP32-C6-MINI-1"
+		(property "Value" "ESP32-C6-MINI-1-N4"
 			(at 0 6.9 90)
 			(unlocked yes)
@@
 			)
 		)
-		(property "Value" "3.3k"
+		(property "Value" "5.1k"
 			(at 0 1.65 0)
 			(layer "F.Fab")
@@
 			)
 		)
-		(property "Value" "SS14 BOOST -> UNNI_AC"
+		(property "Value" "SS14"
 			(at 0 2.6 0)
 			(layer "F.Fab")
