File: unni-smartification-c6/experimental/unni-smartification-c6-10.99-constraints.kicad_pcb (KiCad board)
At the start: 2 copper layers, 83.3 x 65 mm, 72 parts, among them J1 USB-C (replacement daughterbo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, J10 UART TEST, J2 Li-Ion 1S JST-PH, J20 CO2 tap: SDA/SCL/GND, J21 RT/RH tap: RT/RH/GND, J22 TOUCH / LED+ / LED- / GND, J4 UNNI DC / battery input - AC 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, Q1 AO3401A, Q10 AO3400A touch emulator, Q2 AO3401A, Q3 AO3400A, Q4 AO3400A, U1 MCP73831T-2ACI/OT, U10 ESP32-C6-MINI-1, U2 TPS63031DSK, U3 TPS613222ADBZ (5V)

Commit message: Combine USB and ESP boards in KiCad 10.99 layout
Parts:
- removed J10: UART TEST, Connector_JST:JST_XH_S3B-XH-A_1x03_P2.50mm_Horizontal
- removed L1: 1.5uH, Inductor_SMD:L_TDK_NLV32_3.2x2.5mm
- removed L2: 2.2uH, Inductor_SMD:L_TDK_NLV32_3.2x2.5mm
- added D1: SS14, Diode_SMD:D_SMA, F.Cu at (171.1, 61.2)
- added D2: SS14 DNP, Diode_SMD:D_SMA, F.Cu at (171.1, 65.8)
- added J3: UNNI AC / 5V input, Connector_JST:JST_XH_B2B-XH-A_1x02_P2.50mm_Vertical, F.Cu at (170.5, 46.7)
- added Q2: AO3401A, Package_TO_SOT_SMD:SOT-23, F.Cu at (178.9, 60.1)
- added Q4: AO3400A, Package_TO_SOT_SMD:SOT-23, F.Cu at (178.9, 69.0)
- added R12: 220k, Resistor_SMD:R_0603_1608Metric, F.Cu at (186.5, 52.1)
- added R6: 1M, Resistor_SMD:R_0603_1608Metric, F.Cu at (182.5, 49.6)
- added R9: 100k, Resistor_SMD:R_0603_1608Metric, F.Cu at (186.5, 47.1)
- J2: footprint Connector_JST:JST_PH_S2B-PH-K_1x02_P2.00mm_Horizontal -> Connector_JST:JST_PH_B2B-PH-K_1x02_P2.00mm_Vertical
- J20, J21: footprint Connector_JST:JST_XH_S3B-XH-A_1x03_P2.50mm_Horizontal -> Connector_JST:JST_XH_B3B-XH-A_1x03_P2.50mm_Vertical
- J22: footprint Connector_JST:JST_XH_S4B-XH-A_1x04_P2.50mm_Horizontal -> Connector_JST:JST_XH_B4B-XH-A_1x04_P2.50mm_Vertical
- J4: value UNNI DC / battery input - AC / 5V Input -> UNNI DC / battery input; footprint Connector_JST:JST_XH_S3B-XH-A_1x03_P2.50mm_Horizontal -> Connector_JST:JST_XH_B2B-XH-A_1x02_P2.50mm_Vertical
- moved H4 256.1 mm to (239.2, 91.7)
- moved H3 249.7 mm to (232.2, 91.9)
- moved J1 247.1 mm to (233.2, 81.9), turned to 180 degrees
- moved H2 242.0 mm to (224.2, 91.2)
- moved R2 241.2 mm to (225.8, 84.8)
- moved H1 241.0 mm to (224.7, 87.2)
- moved R1 240.3 mm to (225.8, 82.3)
- moved D1 218.0 mm to (194.4, 98.7)
- moved Q4 214.5 mm to (192.8, 94.2)
- moved Q2 212.6 mm to (192.8, 89.7)
- moved R13 211.9 mm to (187.9, 97.8)
- moved R12 210.5 mm to (187.9, 94.9)
- moved R9 209.2 mm to (187.9, 91.9)
- moved R6 207.9 mm to (187.9, 89.0)
- moved U1 204.1 mm to (196.3, 55.8)
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Connections:
- J4 pad 2: UNNI_AC -> GND
- R7 pad 1: Net-(Q2-G) -> +BATT
- R7 pad 2: +BATT -> Net-(Q2-G)
Routing:
- removed copper zone on F.Cu, net +3V3
- removed copper zone on F.Cu, net +5V
- removed copper zone on F.Cu, net /USB + Power/BOOST_IN
- removed copper zone on B.Cu, net GND
- removed copper zone on F.Cu, net GND
- removed copper zone on F.Cu, net SYS
Other:
- board size 83.3 x 65 mm -> 19 x 18 mm
- board text removed: "ESP / INTERFACE BOARD 46 x 32 mm MAX"
- board text removed: "TOP DATUM / USB"
- board text removed: "USB / POWER BOARD 19 x <=65 mm"

Commit message: Add BOM Metadata, iBom, fix validation, pcbway order
this is the state the PCBs were ordered at PCBWay.com

Thank you PCBWay for sponsoring the boards for this ridicoulus project!
Parts:
- C32: value 220pF DNP -> 220pF
- D3: value SS14 USB -> UNNI_AC -> SS14
- D4: value SS14 BOOST -> UNNI_AC -> SS14
- J1: value USB-C (replacement daughterboard) -> UJ20-C-H-G-SMT-1-P16-TR
- J2: value Li-Ion 1S JST-PH -> B2B-PH-K-S
- J3: value UNNI AC / 5V input -> B6B-PH-K-S
- J4: value UNNI DC / battery input -> S3B-PH-SM4-TB
- Q10: value AO3400A touch emulator -> AO3400A
- R3: value 3.3k -> 5.1k
- R9: value 100k -> 1M
- U1: value MCP73831T-2ACI/OT -> MCP73831
- U10: value ESP32-C6-MINI-1 -> ESP32-C6-MINI-1-N4
- U2: value TPS63031DSK -> TPS63031
- U3: value TPS613222ADBZ (5V) -> TPS613222A
Changed lines of the file:
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@@
 			)
 		)
-		(property "Value" "UNNI DC / battery input"
+		(property "Value" "S3B-PH-SM4-TB"
 			(at 1.25 4.6 0)
 			(layer "F.Fab")
@@
 			)
 		)
-		(property "Value" "TPS63031DSK"
+		(property "Value" "TPS63031"
 			(at 0 2.2 0)
 			(layer "F.Fab")
@@
 			)
 		)
-		(property "Value" "UNNI AC / 5V input"
+		(property "Value" "B6B-PH-K-S"
 			(at 1.25 4.6 0)
 			(layer "F.Fab")
@@
 			)
 		)
-		(property "Value" "TPS613222ADBZ (5V)"
+		(property "Value" "TPS613222A"
 			(at 0 2.4 0)
 			(layer "F.Fab")
@@
 			)
 		)
-		(property "Value" "100k"
+		(property "Value" "1M"
 			(at 0 1.43 0)
 			(layer "F.Fab")
@@
 			)
 		)
-		(property "Value" "SS14 USB -> UNNI_AC"
+		(property "Value" "SS14"
 			(at 0 2.6 0)
 			(layer "F.Fab")
@@
 			)
 		)
-		(property "Value" "Li-Ion 1S JST-PH"
+		(property "Value" "B2B-PH-K-S"
 			(at 1 4 0)
 			(layer "F.Fab")
@@
 			)
 		)
-		(property "Value" "USB-C (replacement daughterboard)"
+		(property "Value" "UJ20-C-H-G-SMT-1-P16-TR"
 			(at 0 5 180)
 			(unlocked yes)
@@
 			)
 		)
-		(property "Value" "220pF DNP"
+		(property "Value" "220pF"
 			(at 0 1.43 90)
 			(layer "F.Fab")
@@
 			)
 		)
-		(property "Value" "AO3400A touch emulator"
+		(property "Value" "AO3400A"
 			(at 0 2.4 90)
 			(layer "F.Fab")
@@
 			)
 		)
-		(property "Value" "MCP73831T-2ACI/OT"
+		(property "Value" "MCP73831"
 			(at 0 2.4 0)
 			(layer "F.Fab")
@@
 			)
 		)
-		(property "Value" "ESP32-C6-MINI-1"
+		(property "Value" "ESP32-C6-MINI-1-N4"
 			(at 0 6.9 90)
 			(unlocked yes)
@@
 			)
 		)
-		(property "Value" "3.3k"
+		(property "Value" "5.1k"
 			(at 0 1.65 0)
 			(layer "F.Fab")
@@
 			)
 		)
-		(property "Value" "SS14 BOOST -> UNNI_AC"
+		(property "Value" "SS14"
 			(at 0 2.6 0)
 			(layer "F.Fab")
